File: rotaryEncoderWith595/rotaryEncoderWith595.kicad_pcb (KiCad board)
At the start: 2 copper layers, 68 parts, among them J1 OUTCON, SW1 ROTENC, SW2 ROTENC, SW3 ROTENC, SW4 ROTENC, SW5 IN, SW6 IN, SW7 IN, SW8 IN, U1 74HC165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

Commit message: finish route
Parts:
- moved D3 21.3 mm to (92.7, 88.0)
- moved D4 21.3 mm to (92.7, 82.4)
- moved D6 21.3 mm to (92.7, 71.0)
- moved D7 21.3 mm to (92.7, 65.5)
- moved D8 21.3 mm to (92.7, 59.9)
- moved D1 21.3 mm to (92.7, 99.0)
- moved D2 21.3 mm to (92.7, 93.5)
- moved D5 21.3 mm to (92.7, 76.5)
- moved C1 15.3 mm to (117.8, 87.0), turned to 180 degrees
- moved D12 8.56 mm to (199.3, 77.2)
- moved D16 8.56 mm to (199.3, 99.2)
- moved D10 8.56 mm to (199.3, 66.0)
- moved D11 8.56 mm to (199.3, 71.6)
- moved D13 8.56 mm to (199.3, 82.5)
- moved D14 8.56 mm to (199.3, 88.0)
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Connections:
- J1 pad 1: /OUT165 -> /CLK165
- J1 pad 3: /CLK165 -> GND
- J1 pad 4: /RCLK595 -> +5V
- J1 pad 6: /SER595 -> /RCLK595
- J1 pad 7: +5V -> /SER595
- J1 pad 8: GND -> /OUT165
Routing:
- net GND: track 456.8 -> 807.8 mm, vias 6 -> 10
- net /CLK165: track 20.5 -> 281.3 mm, vias 0 -> 4
- net +5V: track 207.4 -> 406.5 mm, vias 6 -> 10
- net /LD165: track 85.3 -> 270.9 mm, vias 0 -> 2
- net Net-(U1-Q7): track 16.0 -> 178.6 mm, vias 0 -> 2
- net /OUT165: track 0.00 -> 90.4 mm
- net Net-(D1-A): track 0.00 -> 34.8 mm
- net Net-(D2-A): track 0.00 -> 31.0 mm
- net Net-(D3-A): track 0.00 -> 29.5 mm
- net Net-(D4-A): track 0.00 -> 28.9 mm
- net /SRCLK595: track 35.3 -> 63.7 mm, vias 0 -> 2
- net Net-(D5-A): track 0.00 -> 28.2 mm
- net Net-(D6-A): track 0.00 -> 27.5 mm
- net Net-(D7-A): track 0.00 -> 26.9 mm
- net /RCLK595: track 35.3 -> 62.1 mm
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
Commit message: finish route and generate pdf
Parts:
- added H1: MountingHole_Pad, MountingHole:MountingHole_3mm_Pad, F.Cu at (211.0, 52.5)
- added H2: MountingHole_Pad, MountingHole:MountingHole_3mm_Pad, F.Cu at (94.0, 136.0)
- added H3: MountingHole_Pad, MountingHole:MountingHole_3mm_Pad, F.Cu at (94.0, 110.0)
- added H4: MountingHole_Pad, MountingHole:MountingHole_3mm_Pad, F.Cu at (211.0, 99.5)
- added REF**: CE-Logo_11.2x8mm_SilkScreen, Symbol:CE-Logo_11.2x8mm_SilkScreen, F.Cu at (107.5, 136.0)
- added REF**: KiCad-Logo_8mm_SilkScreen, Symbol:KiCad-Logo_8mm_SilkScreen, F.Cu at (149.0, 136.0)
- moved J1 12.1 mm to (136.1, 58.0)
- moved C4 1.03 mm to (142.8, 62.0)
Connections:
- J1 pad 1: /CLK165 -> GND
- J1 pad 2: /LD165 -> +5V
- J1 pad 3: GND -> /CLK165
- J1 pad 4: +5V -> /LD165
- J1 pad 7: /SER595 -> /OUT165
- J1 pad 8: /OUT165 -> /SER595
Routing:
- net GND: track 807.8 -> 781.9 mm
- net /OUT165: track 90.4 -> 105.7 mm
- net /RCLK595: track 62.1 -> 54.7 mm
- net /CLK165: track 281.3 -> 274.4 mm
- net /SER595: track 22.4 -> 29.2 mm
- net /SRCLK595: track 63.7 -> 57.1 mm
- net /LD165: track 270.9 -> 268.8 mm, vias 2 -> 4
- net +5V: track 406.5 -> 408.0 mm, vias 10 -> 8
Other:
- board outline added: 130 x 95 mm
- board text added: "2024"
- board text added: "27 JUNI 2024 18:04"
- board text added: "GND 5V CLK165 LD165 SRCLK595 RCLK595 OUT165 SER595"
