File: rotaryEncoderWith595/rotaryEncoderWith595.kicad_sch (KiCad schematic)
At the start: 68 parts, among them J1 OUTCON, SW1 ROTENC, SW2 ROTENC, SW3 ROTENC, SW4 ROTENC, SW5 IN, SW6 IN, SW7 IN, SW8 IN, U1 74HC165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

Commit message: finish route
Connections:
- net +5V: now also J1.4 (Pin_4); no longer J1.7 (Pin_7)
- net CLK165: now also J1.1 (Pin_1); no longer J1.3 (Pin_3)
- net GND: now also J1.3 (Pin_3); no longer J1.8 (Pin_8)
- net OUT165: now also J1.8 (Pin_8); no longer J1.1 (Pin_1)
- net RCLK595: now also J1.6 (Pin_6); no longer J1.4 (Pin_4)
- net SER595: now also J1.7 (Pin_7); no longer J1.6 (Pin_6)

Commit message: finish route and generate pdf
Parts:
- added H1, H2, H3, H4: MountingHole_Pad, MountingHole:MountingHole_3mm_Pad, symbol Mechanical:MountingHole_Pad
Connections:
- net +5V: now also J1.2 (Pin_2); no longer J1.4 (Pin_4)
- net CLK165: now also J1.3 (Pin_3); no longer J1.1 (Pin_1)
- net GND: now also J1.1 (Pin_1); no longer J1.3 (Pin_3)
- net LD165: now also J1.4 (Pin_4); no longer J1.2 (Pin_2)
- net OUT165: now also J1.7 (Pin_7); no longer J1.8 (Pin_8)
- net SER595: now also J1.8 (Pin_8); no longer J1.7 (Pin_7)
- no-connect marks 4 -> 8

Commit message: add schematic svg
Other:
- note added: "74HC165"
- note added: "74HC595"
- note added: "Input, Rotary Encoder and Breakout"
- company: (none) -> AHAH - Crumbs
- title: (none) -> 4 Input 4 Rotary Encoder 
- moved on the sheet: C1, C10, C11, C12, C2, C3, C4, C5, C6, C7, C8, C9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
