File: black-magic-103rc/black-magic-103rc.kicad_sch (KiCad schematic)
At the start: 29 parts, among them J1 USB_B_Micro, Q1 DMG1024UV, Q2 DMG1023UV, SW1 SW_SPST, U1 USBLC6-2P6, U2 SN74LVC2T45DCUR, U3 STM32F103RCTx, U4 AMS1117-3.3, Y1 8MHz

Commit message: [01-16-1532] very little schematic update
Parts:
- added C11, C12, C13, C14, C15, C16, C17, C18: 100n, symbol Device:C
- added U5, U6, U7: SN74LVC2T45DCUR, Package_SO:VSSOP-8_2.4x2.1mm_P0.5mm, symbol Logic_LevelTranslator:SN74LVC2T45DCUR
Connections:
- net +3.3V: now also U2.1 (VCCA), C11.1, C13.1, C15.1, C16.1, U5.1 (VCCA), U6.1 (VCCA), U7.1 (VCCA)
- net GND: now also U2.4 (GND), C11.2, C12.2, C13.2, C14.2, C15.2, C16.2, C17.2, C18.2, U5.4 (GND), U6.4 (GND), U7.4 (GND)
- net at U2.8 (VCCB): now also C12.1
- new net: C14.1, U5.8 (VCCB)
- new net: C17.1, U6.8 (VCCB)
- new net: C18.1, U7.8 (VCCB)
