File: hokushime-hiroshe-usb-to-rs232/hardware/hokushime-hiroshe-usb-to-rs232/hokushime-db9-to-rs232.kicad_pcb (KiCad board)
At the start: 2 copper layers, 52.4 x 47.7 mm, 39 parts, among them IC1 SP3243EC/EB, J1 Conn1, J2 USB_B, J3 Conn2, U1 FT232BM/BL, U3 93CxxC, Y1 6Mhz

Commit message: [06-13-0759] change package to correct package SSOP and 32QFP, also make manufacture step doc
Parts:
- IC1: footprint Package_SO:TSSOP-28_4.4x9.7mm_P0.65mm -> Package_SO:SSOP-28_5.3x10.2mm_P0.65mm
- U1: footprint Package_QFP:LQFP-48_7x7mm_P0.5mm -> Package_QFP:LQFP-32_7x7mm_P0.8mm
- moved J3 2.63 mm to (177.1, 85.2)
- moved TP1 1.58 mm to (159.6, 101.2)
- moved C7 0.98 mm to (163.8, 101.0)
- moved C2 0.92 mm to (163.7, 103.3)
- moved U1 0.28 mm to (146.2, 89.0), turned to 0 degrees
Routing:
- net Net-(U1-XTIN): track 22.5 -> 34.7 mm
- net GND: track 201.8 -> 212.0 mm, vias 16 -> 10
- net /93C66_SCLK: track 4.27 -> 12.2 mm, vias 0 -> 2
- net /TXD: track 7.76 -> 15.0 mm, vias 0 -> 2
- net Net-(U1-AVCC): track 22.7 -> 15.6 mm, vias 0 -> 2
- net /93C66_CS: track 37.6 -> 30.6 mm
- net Net-(JP1-C): track 21.3 -> 15.7 mm, vias 2 -> 0
- net Net-(U1-XTOUT): track 15.4 -> 9.93 mm
- net VBUS: track 50.9 -> 46.5 mm
- net +5V: track 177.6 -> 181.9 mm
- net /~{CTS}: track 13.3 -> 16.7 mm
- net /~{DTR}: track 15.6 -> 18.6 mm, vias 2 -> 0
- net /CONN2_DCD: track 5.30 -> 8.03 mm
- net Net-(U1-~{RSTOUT}): track 9.43 -> 12.1 mm
- net /~{DSR}: track 11.9 -> 14.5 mm
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