File: rp2350a-tempel/rp2350a-tempel.kicad_sch (KiCad schematic)
At the start: 36 parts, among them J1 Conn_North, J2 Conn_East, J3 Conn_South, J4 Conn_West, SW1 BOOT SELECTOR, SW2 RST, U1 AMS1117-3.3, U2 W25Q16JVSS, U3 RP2350_60QFN, Y1 12Mhz HC49-SD

Commit message: feat: finish routing
Update README.md
Parts:
- L1: value L -> 3.3uH
Connections:
- net +3.3V: now also J1.1 (Pin_1); no longer J1.2 (Pin_2)
- net +5V: now also J1.7 (Pin_7); no longer J1.6 (Pin_6)
- net GND: now also J1.6 (Pin_6); no longer J1.7 (Pin_7)
- net GPIO28_ADC2: now also J1.8 (Pin_8); no longer J1.9 (Pin_9)
- net GPIO29_ADC3: now also J1.9 (Pin_9); no longer J1.8 (Pin_8)
- net ~{BOOTSEL}: now also J1.2 (Pin_2); no longer J1.1 (Pin_1)
- no-connect marks 0 -> 1
Other:
- title: (none) -> Tempel RP2350
