File: proto-double-layer-poc/proto-double-layer-poc.kicad_sch (KiCad schematic)
At the start: 41 parts, among them J1 1.47 IPS LCD, J2 USB2UART, Q1 SS8050, Q2 SS8050, SW1 RST, SW2 Boot, SW3 IN1, SW4 IN2, SW5 IN4, SW6 IN4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

Commit message: fix: swapped spid(mosi) in proto-double-layer
Connections:
- net SDA: now also U1.19 (IO11); no longer U1.21 (IO13)
Changed lines of the file:
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@@
-	)
-	(no_connect
-		(at 81.28 110.49)
 	)
 	(no_connect
@@
 	)
 	(no_connect
+		(at 81.28 115.57)
+	)
+	(no_connect
 		(at 163.83 100.33)
 	)
@@
 	(wire
 		(pts
+			(xy 71.12 110.49) (xy 81.28 110.49)
+		)
+		(stroke
+			(width 0)
+			(type default)
+		)
+	)
+	(wire
+		(pts
 			(xy 240.03 72.39) (xy 232.41 72.39)
 		)
@@
 		(pts
 			(xy 191.77 69.85) (xy 186.69 69.85)
-		)
-		(stroke
-			(width 0)
-			(type default)
-		)
-	)
-	(wire
-		(pts
-			(xy 71.12 115.57) (xy 81.28 115.57)
 		)
 		(stroke
@@
 		)
 	)
+	(label "SDA"
+		(at 71.12 110.49 0)
+		(effects
+			(font
+				(size 1.27 1.27)
+			)
+			(justify left bottom)
+		)
+	)
 	(label "CS"
 		(at 90.17 163.83 180)
@@
 		)
 	)
-	(label "SDA"
-		(at 71.12 115.57 0)
-		(effects
-			(font
-				(size 1.27 1.27)
-			)
-			(justify left bottom)
-		)
-	)
