File: proto-double-layer-poc/proto-double-layer-poc.kicad_pcb (KiCad board)
At the start: 2 copper layers, 57.1 x 46.3 mm, 41 parts, among them J1 1.47 IPS LCD, J2 USB2UART, Q1 SS8050, Q2 SS8050, SW1 RST, SW2 Boot, SW3 IN1, SW4 IN2, SW5 IN4, SW6 IN4, U1 ESP32-S3-WROOM-1, U2 CH340C, U4 AMS1117-3.3

Commit message: generating pcb and schematic image
Other:
- board text added: "blk cs dc rst sda sck 3.3 gnd"
