File: rp2350-dev-board/rp2350-dev-board.kicad_sch (KiCad schematic)
At the start: 91 parts, among them J1 USB_C_Receptacle_USB2.0_14P, J13 PWR_IN, J14 SWD, J15 TMC2209_VIN, J16 TMC2209_Conn, J17 Conn_West, J18 Conn_North, J19 Conn_South, J20 Conn_East, J3 HDMI_A, J4 MS1, J5 MS2, J6 Spread, J7 DriverConn, J8 1.47_IPS_LCD, SW1 BTN1, SW2 BTN1, SW3 BTN1, SW4 BTN1, SW5 BTN1, SW6 BOOT SELECTOR, SW7 RST, U4 L7805, U6 TMC2209-LA, U7 W25Q16JVSS, U8 AMS1117-3.3, U9 RP2350_60QFN, Y1 12Mhz HC49-SD

Commit message: feat(rp2350-dev-board): routing phase 1
Connections:
- net GPIO28_ADC2: now also J18.9 (Pin_9); no longer J18.8 (Pin_8)
- net GPIO29_ADC3: now also J18.8 (Pin_8); no longer J18.9 (Pin_9)
- net USB_DM: no longer J18.5 (Pin_5)
- net USB_DP: no longer J18.4 (Pin_4)
- net ~{BOOTSEL}: now also J18.5 (Pin_5); no longer J18.2 (Pin_2)
- no-connect marks 12 -> 14
Changed lines of the file:
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@@
 	)
 	(no_connect
+		(at 341.63 59.69)
+	)
+	(no_connect
 		(at 41.91 66.04)
 	)
 	(no_connect
+		(at 346.71 59.69)
+	)
+	(no_connect
 		(at 58.42 132.08)
 	)
@@
 	(wire
 		(pts
-			(xy 222.25 34.29) (xy 222.25 35.56)
+			(xy 359.41 44.45) (xy 359.41 59.69)
 		)
 		(stroke
@@
 	(wire
 		(pts
-			(xy 148.59 168.91) (xy 161.29 168.91)
+			(xy 222.25 34.29) (xy 222.25 35.56)
 		)
 		(stroke
@@
 	(wire
 		(pts
-			(xy 223.52 264.16) (xy 223.52 261.62)
+			(xy 148.59 168.91) (xy 161.29 168.91)
 		)
 		(stroke
@@
 	(wire
 		(pts
-			(xy 359.41 107.95) (xy 359.41 97.79)
+			(xy 223.52 264.16) (xy 223.52 261.62)
 		)
 		(stroke
@@
 	(wire
 		(pts
-			(xy 181.61 33.02) (xy 181.61 31.75)
+			(xy 359.41 107.95) (xy 359.41 97.79)
 		)
 		(stroke
@@
 	(wire
 		(pts
-			(xy 231.14 36.83) (xy 228.6 36.83)
+			(xy 181.61 33.02) (xy 181.61 31.75)
 		)
 		(stroke
@@
 	(wire
 		(pts
-			(xy 160.02 86.36) (xy 146.05 86.36)
+			(xy 231.14 36.83) (xy 228.6 36.83)
 		)
 		(stroke
@@
 	(wire
 		(pts
-			(xy 349.25 50.8) (xy 349.25 59.69)
+			(xy 160.02 86.36) (xy 146.05 86.36)
 		)
 		(stroke
@@
 	(wire
 		(pts
-			(xy 346.71 50.8) (xy 346.71 59.69)
-		)
-		(stroke
-			(width 0)
-			(type default)
-		)
-	)
-	(wire
-		(pts
 			(xy 77.47 172.72) (xy 77.47 170.18)
 		)
@@
 	(wire
 		(pts
-			(xy 359.41 44.45) (xy 359.41 59.69)
-		)
-		(stroke
-			(width 0)
-			(type default)
-		)
-	)
-	(wire
-		(pts
 			(xy 356.87 214.63) (xy 356.87 215.9)
 		)
@@
 	(wire
 		(pts
-			(xy 356.87 44.45) (xy 356.87 59.69)
-		)
-		(stroke
-			(width 0)
-			(type default)
-		)
-	)
-	(wire
-		(pts
 			(xy 48.26 96.52) (xy 58.42 96.52)
 		)
@@
 	(wire
 		(pts
-			(xy 341.63 50.8) (xy 341.63 59.69)
-		)
-		(stroke
-			(width 0)
-			(type default)
-		)
-	)
-	(wire
-		(pts
 			(xy 311.15 25.4) (xy 311.15 26.67)
 		)
@@
 	(wire
 		(pts
+			(xy 349.25 50.8) (xy 349.25 59.69)
+		)
+		(stroke
+			(width 0)
+			(type default)
+		)
+	)
+	(wire
+		(pts
 			(xy 63.5 265.43) (xy 63.5 262.89)
 		)
@@
 	(wire
 		(pts
+			(xy 356.87 44.45) (xy 356.87 59.69)
+		)
+		(stroke
+			(width 0)
+			(type default)
+		)
+	)
+	(wire
+		(pts
 			(xy 226.06 251.46) (xy 224.79 251.46)
 		)
@@
 		)
 	)
-	(label "USB_DP"
-		(at 346.71 50.8 270)
-		(effects
-			(font
-				(size 1.27 1.27)
-			)
-			(justify right bottom)
-		)
-	)
 	(label "GPIO16"
 		(at 48.26 96.52 0)
@@
 		)
 	)
+	(label "GPIO29_ADC3"
+		(at 356.87 44.45 270)
+		(effects
+			(font
+				(size 1.27 1.27)
+			)
+			(justify right bottom)
+		)
+	)
 	(label "GPIO19"
 		(at 384.81 85.09 180)
@@
 		)
 	)
-	(label "GPIO28_ADC2"
-		(at 356.87 44.45 270)
-		(effects
-			(font
-				(size 1.27 1.27)
-			)
-			(justify right bottom)
-		)
-	)
 	(label "SPI_SD0"
 		(at 160.02 86.36 180)
@@
 		)
 	)
+	(label "~{BOOTSEL}"
+		(at 349.25 50.8 270)
+		(effects
+			(font
+				(size 1.27 1.27)
+			)
+			(justify right bottom)
+		)
+	)
 	(label "MS2/AD1"
 		(at 78.74 260.35 180)
@@
 		)
 	)
-	(label "~{BOOTSEL}"
-		(at 341.63 50.8 270)
-		(effects
-			(font
-				(size 1.27 1.27)
-			)
-			(justify right bottom)
-		)
-	)
 	(label "SPI_SD3"
 		(at 209.55 81.28 0)
@@
 		)
 	)
+	(label "GPIO28_ADC2"
+		(at 359.41 44.45 270)
+		(effects
+			(font
+				(size 1.27 1.27)
+			)
+			(justify right bottom)
+		)
+	)
 	(label "GPIO1"
 		(at 300.99 60.96 180)
@@
 		)
 	)
-	(label "GPIO29_ADC3"
-		(at 359.41 44.45 270)
-		(effects
-			(font
-				(size 1.27 1.27)
-			)
-			(justify right bottom)
-		)
-	)
 	(label "GPIO26_ADC0"
 		(at 377.19 224.79 90)
@@
 		(effects
 			(font
-				(size 1.27 1.27)
-			)
-			(justify right bottom)
-		)
-	)
-	(label "USB_DM"
-		(at 349.25 50.8 270)
-		(effects
-			(font
