File: miolari/miolari-esp32/miolari-esp32.kicad_pcb (KiCad board)
At the start: 2 copper layers, 105.5 x 66 mm, 63 parts, among them CN1 XT60PW-M, J1 USB2UART, J2 USB2UART, J3 lcd jumper, J4 lcd jumper, J5 lcd jumper, J6 1.47 IPS LCD, J7 ConnBattery, J8 MainConnector, Q1 SS8050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

Commit message: miolari rp2350a routing phase2
Connections:
- R7 pad 1: /USB_DP -> /USB_DM
- R8 pad 1: /USB_DM -> /USB_DP
Routing:
- net /USB_DM: track 64.7 -> 61.8 mm
- net /USB_DP: track 51.9 -> 53.9 mm
- net /DC: track 197.3 -> 198.4 mm
- net VBUS: track 210.3 -> 211.4 mm
