File: miolari/miolari-esp32/miolari-esp32.kicad_sch (KiCad schematic)
At the start: 0 parts

Commit message: miolari finish routing
Parts:
- added C1, C3, C5, C6, C7: 10uF, Capacitor_SMD:C_0805_2012Metric_Pad1.18x1.45mm_HandSolder, symbol Device:C
- added C10, C15: 1uF, Capacitor_SMD:C_0805_2012Metric_Pad1.18x1.45mm_HandSolder, symbol Device:C
- added C11, C13, C4, C9: 100nF, Capacitor_SMD:C_0805_2012Metric_Pad1.18x1.45mm_HandSolder, symbol Device:C
- added C14: 22uF, Capacitor_SMD:C_0805_2012Metric_Pad1.18x1.45mm_HandSolder, symbol Device:C
- added C16, C17: 4.7uF, Capacitor_SMD:C_0805_2012Metric_Pad1.18x1.45mm_HandSolder, symbol Device:C
- added C2: 0.1uF, Capacitor_SMD:C_0805_2012Metric_Pad1.18x1.45mm_HandSolder, symbol Device:C
- added CN1: XT60PW-M, easyeda2kicad:CONN-TH_XT60PW-M, symbol easyeda2kicad:XT60PW-M
- added D1: VDD, LED_SMD:LED_1206_3216Metric_Pad1.42x1.75mm_HandSolder, symbol Device:LED
- added D2: Indicator, LED_SMD:LED_1206_3216Metric_Pad1.42x1.75mm_HandSolder, symbol Device:LED
- added D3: green, LED_SMD:LED_0805_2012Metric_Pad1.15x1.40mm_HandSolder, symbol Device:LED
- added D4: red, LED_SMD:LED_0805_2012Metric_Pad1.15x1.40mm_HandSolder, symbol Device:LED
- added H1, H2, H3, H4: MountingHole, MountingHole:MountingHole_2mm, symbol Mechanical:MountingHole
- added J1, J2: USB2UART, Connector_USB:USB_C_Receptacle_GCT_USB4110, symbol Connector:USB_C_Receptacle_USB2.0_14P
- added J3, J4, J5: lcd jumper, Connector_PinHeader_2.54mm:PinHeader_1x08_P2.54mm_Vertical, symbol Connector_Generic:Conn_01x08
- added J6: 1.47 IPS LCD, Connector_PinHeader_2.54mm:PinHeader_1x08_P2.54mm_Vertical, symbol Connector_Generic:Conn_01x08
- added J7: ConnBattery, Connector_PinHeader_2.54mm:PinHeader_1x03_P2.54mm_Vertical, symbol Connector_Generic:Conn_01x03
- added J8: MainConnector, Connector_IDC:IDC-Header_2x20_P2.54mm_Vertical, symbol Connector_Generic:Conn_02x20_Odd_Even
- added L1: 22uH 1A, Inductor_SMD:L_Bourns_SRP7028A_7.3x6.6mm, symbol Device:L
- added Q1, Q2: SS8050, Package_TO_SOT_SMD:SOT-23_Handsoldering, symbol Transistor_BJT:BC817
- added R1, R14, R18, R19: 1k, Resistor_SMD:R_0805_2012Metric_Pad1.20x1.40mm_HandSolder, symbol Device:R_US
- added R10, R9: 10k, Resistor_SMD:R_0805_2012Metric_Pad1.20x1.40mm_HandSolder, symbol Device:R_US
- added R17: 46.4K, Resistor_SMD:R_0805_2012Metric_Pad1.20x1.40mm_HandSolder, symbol Device:R_US
- added R2: 100, Resistor_SMD:R_0805_2012Metric_Pad1.20x1.40mm_HandSolder, symbol Device:R_US
- added R20: 2K2, Resistor_SMD:R_0805_2012Metric_Pad1.20x1.40mm_HandSolder, symbol Device:R_US
- added R21: 1.13k, Resistor_SMD:R_0805_2012Metric_Pad1.20x1.40mm_HandSolder, symbol Device:R_US
- added R22, R23: 4K7, Resistor_SMD:R_0805_2012Metric_Pad1.20x1.40mm_HandSolder, symbol Device:R_US
- added R24, R25: 1K5, Resistor_SMD:R_0805_2012Metric_Pad1.20x1.40mm_HandSolder, symbol Device:R_US
- added R3, R4, R5, R6: 5K1, Resistor_SMD:R_0805_2012Metric_Pad1.20x1.40mm_HandSolder, symbol Device:R_US
- added R7, R8: 22 / 33, Resistor_SMD:R_0805_2012Metric_Pad1.20x1.40mm_HandSolder, symbol Device:R_US
- added SW1: RST, Button_Switch_SMD:SW_SPST_EVQP7A, symbol Switch:SW_Push
- added SW2: Boot, Button_Switch_SMD:SW_SPST_EVQP7A, symbol Switch:SW_Push
- added U1: USBLC6-2P6, Package_TO_SOT_SMD:SOT-666, symbol Power_Protection:USBLC6-2P6
- added U2: TPS63001_SEPIC_3V3, Package_SON:Texas_DRC0010J_ThermalVias, symbol Regulator_Switching:TPS63001
- added U3: CH340C, Package_SO:SOIC-16_3.9x9.9mm_P1.27mm, symbol Interface_USB:CH340C
- added U4: L7805, Package_TO_SOT_THT:TO-220-3_Horizontal_TabUp, symbol Regulator_Linear:L7805
- added U6: BQ24075RGT_DPPM, Package_DFN_QFN:VQFN-16-1EP_3x3mm_P0.5mm_EP1.6x1.6mm, symbol Battery_Management:BQ24075RGT
- added U7: ESP32-S3-WROOM-1, RF_Module:ESP32-S3-WROOM-1, symbol RF_Module:ESP32-S3-WROOM-1
Connections:
- new net: Q1.1 (B), R9.1
- new net: D2.2 (A), R18.1
- new net: J3.1 (Pin_1), J4.1 (Pin_1)
- new net: J3.2 (Pin_2), J4.2 (Pin_2)
- new net: J3.3 (Pin_3), J4.3 (Pin_3)
- new net: J3.4 (Pin_4), J4.4 (Pin_4)
- new net: J3.5 (Pin_5), J4.5 (Pin_5)
- new net: J3.6 (Pin_6), J4.6 (Pin_6)
- new net: J3.7 (Pin_7), J4.7 (Pin_7)
- new net: J3.8 (Pin_8), J4.8 (Pin_8)
- new net: D4.2 (A), R25.1
- new net: Q2.1 (B), R10.1
- new net: J1.A6 (D+), J1.B6 (D+), U3.5 (UD+)
- new net: J1.A7 (D-), J1.B7 (D-), U3.6 (UD-)
- new net: C2.1, R2.2, U2.6 (EN), U2.7 (PS/SYNC), U2.8 (VINA)
- new net: J1.A5 (CC1), R3.2
- new net: D1.2 (A), R1.2
- new net: L1.1, U2.2 (L2)
- new net: L1.2, U2.4 (L1)
- new net: D3.2 (A), R24.1
- new net: J1.B5 (CC2), R4.2
- new net: J2.A5 (CC1), R5.2
- new net: J2.A6 (D+), J2.B6 (D+), U1.3 (I/O2)
- new net: J2.A7 (D-), J2.B7 (D-), U1.1 (I/O1)
- new net: J2.B5 (CC2), R6.2
- new net: R8.2, U1.4 (I/O2)
- new net: R7.2, U1.6 (I/O1)
- new net: R18.2, U7.4 (IO4)
- new net +12V: C3.1, CN1.2 (+), J8.40 (Pin_40), U4.1 (IN)
- new net +3.3V: C13.1, C14.1, C15.1, C4.1, C5.1, C6.1, J5.2 (Pin_2), J6.2 (Pin_2), J8.36 (Pin_36), R14.1, R19.1, R22.1, R23.1, U2.1 (VOUT), U2.10 (FB), U3.16 (VCC), U3.4 (V3), U7.2 (3V3)
- new net +BATT: C16.1, J7.1 (Pin_1), U6.2 (BAT), U6.3 (BAT)
- new net BLK: J5.8 (Pin_8), J6.8 (Pin_8), J8.29 (Pin_29), U7.9 (IO16)
- new net CS: J5.7 (Pin_7), J6.7 (Pin_7), J8.17 (Pin_17), U7.18 (IO10)
- new net DC: J5.6 (Pin_6), J6.6 (Pin_6), J8.27 (Pin_27), U7.8 (IO15)
- new net DTR: Q2.2 (E), R9.2, U3.13 (~{DTR})
- new net EN: C9.1, Q1.3 (C), R14.2, SW1.2, U7.3 (EN)
- new net GND: C1.2, C10.2, C11.2, C13.2, C14.2, C15.2, C16.2, C17.2, C2.2, C3.2, C4.2, C5.2, C6.2, C7.2, C9.2, CN1.1 (-), D1.1 (K), D2.1 (K), J1.A1 (GND), J1.A12 (GND), J1.B1 (GND), J1.B12 (GND), J2.A1 (GND), J2.A12 (GND), J2.B1 (GND), J2.B12 (GND), J5.1 (Pin_1), J6.1 (Pin_1), J7.3 (Pin_3), J8.39 (Pin_39), R17.2, R20.2, R21.2, R3.1, R4.1, R5.1, R6.1, SW1.1, SW2.1, U1.2 (GND), U2.11 (PGND), U2.3 (PGND), U2.9 (GND), U3.1 (GND), U4.2 (GND), U6.15 (SYSOFF), U6.17 (VSS), U6.4 (~{CE}), U6.6 (EN1), U6.8 (VSS), U7.1 (GND), U7.40 (GND), U7.41 (GND)
- new net GPOUT: J8.7 (Pin_7), U7.5 (IO5)
- new net I2C_SCL: J8.3 (Pin_3), R23.2, U7.38 (IO2)
- new net I2C_SDA: J8.1 (Pin_1), R22.2, U7.39 (IO1)
- new net ILIM: R20.1, U6.12 (ILIM)
- new net IO0: C11.1, Q2.3 (C), R19.2, SW2.2, U7.27 (IO0)
- new net IO17: J8.35 (Pin_35), U7.10 (IO17)
- new net IO18: J8.37 (Pin_37), U7.11 (IO18)
- new net IO3: J8.5 (Pin_5), U7.15 (IO3)
- new net IO38: J8.2 (Pin_2), U7.31 (IO38)
- new net IO39: J8.4 (Pin_4), U7.32 (IO39)
- new net IO40: J8.6 (Pin_6), U7.33 (IO40)
- new net IO41: J8.8 (Pin_8), U7.34 (IO41)
- new net IO42: J8.10 (Pin_10), U7.35 (IO42)
- new net IO45: J8.12 (Pin_12), U7.26 (IO45)
- new net IO46: J8.14 (Pin_14), U7.16 (IO46)
- new net IO47: J8.16 (Pin_16), U7.24 (IO47)
- new net IO48: J8.18 (Pin_18), U7.25 (IO48)
- new net IO6: J8.9 (Pin_9), U7.6 (IO6)
- new net IO7: J8.11 (Pin_11), U7.7 (IO7)
- new net IO8: J8.13 (Pin_13), U7.12 (IO8)
- new net IO9: J8.15 (Pin_15), U7.17 (IO9)
- new net ISET: R21.1, U6.16 (ISET)
- new net MISO: J8.23 (Pin_23), U7.21 (IO13)
- new net MOSI: J5.4 (Pin_4), J6.4 (Pin_4), J8.19 (Pin_19), U7.19 (IO11)
- new net RESET: J5.5 (Pin_5), J6.5 (Pin_5), J8.25 (Pin_25), U7.22 (IO14)
- new net RTS: Q1.2 (E), R10.2, U3.14 (~{RTS})
- new net RXD0: J8.33 (Pin_33), U3.2 (TXD), U7.36 (RXD0)
- new net SCK: J5.3 (Pin_3), J6.3 (Pin_3), J8.21 (Pin_21), U7.20 (IO12)
- new net TMR: R17.1, U6.14 (TMR)
- new net TS: J7.2 (Pin_2), U6.1 (TS)
- new net TXD0: J8.31 (Pin_31), U3.3 (RXD), U7.37 (TXD0)
- new net USB_DM: R8.1, U7.13 (IO19)
- new net USB_DP: R7.1, U7.14 (IO20)
- new net VBUS: C10.1, C7.1, J1.A4 (VBUS), J1.A9 (VBUS), J1.B4 (VBUS), J1.B9 (VBUS), J2.A4 (VBUS), J2.A9 (VBUS), J2.B4 (VBUS), J2.B9 (VBUS), J8.38 (Pin_38), U1.5 (VBUS), U4.3 (OUT), U6.13 (IN)
- new net VDD: C1.1, C17.1, R1.1, R2.1, R24.2, R25.2, U2.5 (VIN), U6.10 (OUT), U6.11 (OUT), U6.5 (EN2)
- new net ~{CHG}: D4.1 (K), U6.9 (~{CHG})
- new net ~{PGOOD}: D3.1 (K), U6.7 (~{PGOOD})
- no-connect marks 0 -> 14
Other:
- note added: "DPPM"
- note added: "ESP32-S3-WROOM-1"
- note added: "GND VCC SCL SDA RES DC CS BLK"
- note added: "LCD JUMPER"
- note added: "Program Fast-Charge Safety Timer (TMR): RTMR = tMAXCHG / (10 × KTMR ) KTMR = 48 s/kΩ from the electrical characteristics table. RTMR = (6.25 hr × 3600 s/hr) / (10 × 48 s/kΩ) = 46.8 kΩ -> 46.4 kΩ"
- note added: "Program the Fast Charge Current (ISET): RISET = KISET / ICHG KISET = 890 AΩ from the electrical characteristics table. RISET = 890 AΩ / 0.8 A = 1.1125 kΩ -> 1.13 kΩ"
- note added: "SEPIC 3.3V"
- note added: "Serial USB"
- note added: "USB"
- note added: "dynamic power path management"
- note added: "miso - Also known as q, this is the input of the serial stream into the ESP32 mosi - Also known as d, this is the output of the serial stream from the ESP32 sclk - Clock signal. Each data bit is clocked out or in on the positive or negative edge of this signal quadwp - Write Protect signal. Only used for 4-bit (qio/qout) transactions. quadhd - Hold signal. Only used for 4-bit (qio/qout) transacti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"
- title: (none) -> Miolari ESP32S3

Commit message: miolari rp2350a routing phase2
Connections:
- net USB_DM: now also R7.1; no longer R8.1
- net USB_DP: now also R8.1; no longer R7.1
Changed lines of the file:
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@@
-		)
-	)
-	(label "USB_DP"
-		(at 106.68 39.37 180)
-		(effects
-			(font
-				(size 1.27 1.27)
-			)
-			(justify right bottom)
 		)
 	)
@@
 		)
 	)
+	(label "USB_DP"
+		(at 106.68 41.91 180)
+		(effects
+			(font
+				(size 1.27 1.27)
+			)
+			(justify right bottom)
+		)
+	)
 	(label "RXD0"
 		(at 97.79 90.17 180)
@@
 		)
 	)
+	(label "USB_DM"
+		(at 106.68 39.37 180)
+		(effects
+			(font
+				(size 1.27 1.27)
+			)
+			(justify right bottom)
+		)
+	)
 	(label "CS"
 		(at 184.15 73.66 0)
@@
 		)
 	)
-	(label "USB_DM"
-		(at 106.68 41.91 180)
-		(effects
-			(font
-				(size 1.27 1.27)
-			)
-			(justify right bottom)
-		)
-	)
