File: miolari/miolari-rsp2350/miolari-rp2350.kicad_pcb (KiCad board)
At the start: 2 copper layers, 105.5 x 66 mm, 65 parts, among them CN1 XT60PW-M, J2 USB2UART, J3 lcd jumper, J4 lcd jumper, J5 lcd jumper, J6 1.47 IPS LCD, J7 ConnBattery, J8 MainConnector, SW3 BOOT SELECTOR, SW4 RST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

Commit message: miolari rp2350a routing phase2
Parts:
- added L2: 3.3uH, Inductor_SMD:L_0805_2012Metric_Pad1.05x1.20mm_HandSolder, F.Cu at (127.1, 68.2)
- added U5: W25Q16JVSS, Package_SO:SOIC-8_5.3x5.3mm_P1.27mm, F.Cu at (120.9, 62.1)
- moved C19 91.5 mm to (118.9, 87.5)
- moved C22 90.6 mm to (126.5, 87.7), turned to 180 degrees
- moved C24 89.3 mm to (133.6, 73.1)
- moved C25 88.6 mm to (133.6, 74.7)
- moved C26 88.0 mm to (133.6, 76.3)
- moved Y1 87.3 mm to (121.3, 91.6)
- moved C20 86.5 mm to (133.4, 69.1)
- moved C23 81.1 mm to (133.4, 67.4)
- moved C12 78.8 mm to (120.9, 66.7), turned to 180 degrees
- moved C21 78.3 mm to (127.1, 66.4)
- moved R16 75.1 mm to (122.7, 87.4), turned to 180 degrees
- moved U9 72.2 mm to (122.1, 76.8)
- moved R13 70.9 mm to (133.5, 65.5)
- moved C27 63.7 mm to (120.9, 56.1), turned to 90 degrees
- moved C29 63.5 mm to (124.1, 56.1), turned to 90 degrees
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Connections:
- J5 pad 3: /SCK -> /GPIO10
- J5 pad 4: /MOSI -> /GPIO11
- J5 pad 5: /RESET -> /GPIO12
- J5 pad 6: /DC -> /GPIO13
- J5 pad 7: /CS -> /GPIO14
- J5 pad 8: /BLK -> /GPIO15
- J6 pad 3: /SCK -> /GPIO10
- J6 pad 4: /MOSI -> /GPIO11
- J6 pad 5: /RESET -> /GPIO12
- J6 pad 6: /DC -> /GPIO13
- J6 pad 7: /CS -> /GPIO14
- J6 pad 8: /BLK -> /GPIO15
- J8 pad 1: /GPIO0 -> /GPIO19
- J8 pad 10: /GPIO23 -> /GPIO14
- J8 pad 11: /GPIO5 -> /GPIO24
- J8 pad 12: /GPIO24 -> /GPIO13
- J8 pad 13: /GPIO6 -> /GPIO25
- J8 pad 14: /GPIO25 -> /GPIO12
- J8 pad 15: /GPIO7 -> /GPIO26_ADC0
- J8 pad 16: /GPIO26_ADC0 -> /GPIO11
- J8 pad 17: /GPIO8 -> /GPIO27_ADC1
- J8 pad 18: /GPIO27_ADC1 -> /GPIO10
- J8 pad 19: /GPIO9 -> /GPIO28_ADC2
- J8 pad 2: /GPIO19 -> /GPIO18
- J8 pad 20: /GPIO28_ADC2 -> /GPIO9
- J8 pad 21: /GPIO10 -> /GPIO29_ADC3
- J8 pad 22: /GPIO29_ADC3 -> /GPIO8
- J8 pad 23: /GPIO11 -> /SWCLK
- J8 pad 24: /SWCLK -> /GPIO7
- J8 pad 25: /GPIO12 -> /SWD
- J8 pad 26: /SWD -> /GPIO6
- J8 pad 27: /GPIO13 -> unconnected-(J8-Pin_27-Pad27)
- J8 pad 28: unconnected-(J8-Pin_28-Pad28) -> /GPIO5
- J8 pad 29: /GPIO14 -> unconnected-(J8-Pin_29-Pad29)
- J8 pad 3: /GPIO1 -> /GPIO20
- J8 pad 30: unconnected-(J8-Pin_30-Pad30) -> /GPIO4
- J8 pad 31: /GPIO15 -> unconnected-(J8-Pin_31-Pad31)
- J8 pad 32: unconnected-(J8-Pin_32-Pad32) -> /GPIO3
- J8 pad 33: /GPIO16 -> unconnected-(J8-Pin_33-Pad33)
- J8 pad 34: unconnected-(J8-Pin_34-Pad34) -> /GPIO2
- J8 pad 35: /GPIO17 -> +3.3V
- J8 pad 36: +3.3V -> /GPIO1
- J8 pad 37: /GPIO18 -> VBUS
- J8 pad 38: VBUS -> /GPIO0
- J8 pad 39: GND -> +12V
- J8 pad 4: /GPIO20 -> /GPIO17
- J8 pad 40: +12V -> GND
- J8 pad 5: /GPIO2 -> /GPIO21
- J8 pad 6: /GPIO21 -> /GPIO16
- J8 pad 7: /GPIO3 -> /GPIO22
- J8 pad 8: /GPIO22 -> /GPIO15
- J8 pad 9: /GPIO4 -> /GPIO23
- R7 pad 1: /USB_DP -> /USB_DM
- R8 pad 1: /USB_DM -> /USB_DP
Routing:
- net (no net): track 463.8 -> 0.00 mm, vias 5 -> 0
- net /DC: track 197.3 -> 0.00 mm, vias 3 -> 0
- net /BLK: track 165.3 -> 0.00 mm, vias 4 -> 0
- net GND: track 451.0 -> 594.5 mm, vias 0 -> 14
- net /SCK: track 141.3 -> 0.00 mm, vias 2 -> 0
- net /MOSI: track 140.0 -> 0.00 mm, vias 2 -> 0
- net /CS: track 126.3 -> 0.00 mm, vias 2 -> 0
- net +1V1: track 0.00 -> 125.0 mm, vias 0 -> 5
- net /GPIO16: track 142.6 -> 23.7 mm, vias 3 -> 0
- net /RESET: track 118.5 -> 0.00 mm, vias 3 -> 0
- net /GPIO3: track 139.8 -> 46.7 mm, vias 2 -> 0
- net /GPIO19: track 116.8 -> 25.7 mm, vias 2 -> 0
- net /GPIO7: track 125.5 -> 36.6 mm, vias 2 -> 0
- net /GPIO20: track 119.8 -> 32.4 mm, vias 2 -> 0
- net /GPIO4: track 132.3 -> 45.0 mm, vias 2 -> 0
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
Commit message: miolari rp2350a routing phase3
Parts:
- turned C5 to 180 degrees
- turned C6 to 180 degrees
Routing:
- net GND: track 594.5 -> 654.3 mm, vias 14 -> 10
- net VBUS: track 181.7 -> 221.8 mm
- net /GPIO11: track 101.3 -> 127.4 mm, vias 1 -> 2
- net +3.3V: track 360.6 -> 377.7 mm, vias 8 -> 6
- net /GPIO15: track 78.0 -> 94.0 mm
- net /GPIO14: track 81.1 -> 96.6 mm
- net +12V: track 88.2 -> 103.4 mm
- net VDD: track 96.7 -> 108.7 mm
- net +1V1: track 125.0 -> 134.6 mm
- net /~{CHG}: track 7.03 -> 14.0 mm
- net /SWD: track 59.1 -> 54.5 mm
- net /GPIO10: track 87.0 -> 90.5 mm
- net /GPIO2: track 49.5 -> 46.3 mm
- net /GPIO1: track 51.1 -> 47.9 mm
- net /GPIO0: track 52.6 -> 49.4 mm
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