File: temp-measurement-dongle/electronics/production/tmd.kicad_pcb (KiCad board)
At the start: 2 copper layers, 70.3 x 67.5 mm, 73 parts, among them J1 USB2UART, J2 1.47 IPS LCD, J3 ConnBattery, J4 RTD_PT100, Q1 SS8050, Q2 SS8050, Q3 SS8050, SW1 RST, SW2 IN1, SW3 Boot, SW4 IN2, SW5 IN4, SW6 IN4, SW7 IN5, U1 CH340C, U2 ESP32-S3-WROOM-1, U3 TPS63001_SEPIC_3V3, U4 MAX31865xTP, U5 BQ24075RGT_DPPM

Commit message: updated with newer kicad version
Other:
- board size 70.3 x 67.5 mm -> 68.4 x 67.5 mm
