File: temp-measurement-dongle/electronics/prototype/v2/tmd-v2.kicad_sch (KiCad schematic)
At the start: 90 parts, among them J1 USB2UART, J2 1.47 IPS LCD, J3 ConnBattery, J4 RTD_PT100, J5 lcd jumper, J6 lcd jumper, J7 lcd jumper, Q1 SS8050, Q2 SS8050, Q3 SS8050, Q5 SS8050, SW1 RST, SW2 IN1, SW3 Boot, SW4 IN2, SW5 IN4, SW6 IN4, SW7 IN5, SW8 IN6, U1 CH340C, U2 ESP32-S3-WROOM-1, U3 TPS63001_SEPIC_3V3, U4 MAX31865xTP, U5 BQ24075RGT_DPPM, U7 BQ27421YZFR-G1A

Commit message: use pcb shape from solidwork
Parts:
- removed C1, C25, C3, C5, C6, C9: 100nF, Capacitor_SMD:C_0805_2012Metric_Pad1.18x1.45mm_HandSolder, symbol Device:C
- removed J4: RTD_PT100, TerminalBlock_Phoenix:TerminalBlock_Phoenix_PT-1,5-3-5.0-H_1x03_P5.00mm_Horizontal, symbol Connector:Screw_Terminal_01x03
- removed R1, R10, R29, R3, R7, R9: 1k, Resistor_SMD:R_0805_2012Metric_Pad1.20x1.40mm_HandSolder, symbol Device:R_US
- removed R26: 10K, Resistor_SMD:R_0805_2012Metric_Pad1.20x1.40mm_HandSolder, symbol Device:R_US
- removed R28: 10k, Resistor_SMD:R_0805_2012Metric_Pad1.20x1.40mm_HandSolder, symbol Device:R_US
- removed SW2: IN1, keyswitches.pretty-master:Kailh_socket_MX_optional_reversible_platemount, symbol Switch:SW_Push
- removed SW4: IN2, keyswitches.pretty-master:Kailh_socket_MX_optional_reversible_platemount, symbol Switch:SW_Push
- removed SW5, SW6: IN4, keyswitches.pretty-master:Kailh_socket_MX_optional_reversible_platemount, symbol Switch:SW_Push
- removed SW7: IN5, keyswitches.pretty-master:Kailh_socket_MX_optional_reversible_platemount, symbol Switch:SW_Push
- removed SW8: IN6, keyswitches.pretty-master:Kailh_socket_MX_optional_reversible_platemount, symbol Switch:SW_Push
- added C26: 100nF, Capacitor_SMD:C_0805_2012Metric_Pad1.18x1.45mm_HandSolder, symbol Device:C
- added J8: RTD_PT100, Connector_PinHeader_2.54mm:PinHeader_1x03_P2.54mm_Horizontal, symbol Connector_Generic:Conn_01x03
- added R30, R31, R32: 1k, Resistor_SMD:R_0805_2012Metric_Pad1.20x1.40mm_HandSolder, symbol Device:R_US
- added SW9: PS Joystick, easyeda2kicad:SW-TH_RKJXV1224005, symbol easyeda2kicad:RKJXV1224005
- J6, J7: footprint Connector_PinHeader_2.54mm:PinHeader_1x08_P2.54mm_Vertical -> Connector_PinHeader_2.54mm:PinHeader_1x08_P2.54mm_Horizontal
- R24: value 10k -> 200
- R25: value 10K -> 200
Connections:
- net +3.3V: now also R32.1, SW9.3 (A), SW9.4 (A); no longer R24.1
- net GND: now also C26.2, R30.1, R31.2, SW9.d; no longer R25.2
- net ~{CHG}: no longer Q3.1 (B)
- net at C12.1, Q3.2 (E), U2.31 (IO38): no longer R25.1
- net at U7.A1 (GPOUT): now also R25.2; no longer Q5.1 (B)
- net at C20.2, U4.8 (RTDIN-), U4.9 (FORCE-): now also J8.3 (Pin_3)
- net at C20.1, JP2.1 (A), U4.7 (RTDIN+): now also J8.2 (Pin_2)
- net at JP1.1 (A), JP2.2 (B), U4.5 (FORCE+): now also J8.1 (Pin_1)
- net IN1 renamed AN2
- net AN2: now also SW9.5 (DTA)
- net IN2 renamed AN1
- net AN1: now also SW9.2 (DTA)
- net IN3 renamed ANSW
- net ANSW: now also C26.1, R32.2, SW9.c
- net IN4: no longer names the net of U2.14 (IO20)
- net IN5: no longer names the net of U2.23 (IO21)
- net IN6: no longer names the net of U2.33 (IO40)
- new net: Q3.1 (B), R24.1
- new net: R30.2, SW9.1 (B)
- new net: R31.1, SW9.6 (B)
- new net: Q5.1 (B), R25.1
- no-connect marks 18 -> 27
Other:
- note added: "Analog"
- note added: "Excluded From Board"
- moved on the sheet: C24, H1, H2, H3, H4, Q5, R27

Commit message: complete tmd v2 routing
Parts:
- J3: footprint Connector_PinHeader_2.54mm:PinHeader_1x03_P2.54mm_Vertical -> Connector_PinHeader_2.54mm:PinHeader_1x03_P2.54mm_Horizontal
- J6: footprint Connector_PinHeader_2.54mm:PinHeader_1x08_P2.54mm_Horizontal -> Connector_PinHeader_2.54mm:PinHeader_1x08_P2.54mm_Vertical
Changed lines of the file:
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@@
 			)
 		)
-		(property "Footprint" "Connector_PinHeader_2.54mm:PinHeader_1x08_P2.54mm_Horizontal"
+		(property "Footprint" "Connector_PinHeader_2.54mm:PinHeader_1x08_P2.54mm_Vertical"
 			(at 175.26 152.4 0)
 			(hide yes)
@@
 			)
 		)
-		(property "Footprint" "Connector_PinHeader_2.54mm:PinHeader_1x03_P2.54mm_Vertical"
+		(property "Footprint" "Connector_PinHeader_2.54mm:PinHeader_1x03_P2.54mm_Horizontal"
 			(at 308.61 48.26 0)
 			(hide yes)
