File: realtime-communication/hardware/rt_hw_v1/BQ27441_Batt_Fuel_Gauge.kicad_sch (KiCad schematic)
At the start: 9 parts, among them J2 BattConn, U4 BQ27441-G1

Commit message: add regular sdcard to rt board
Parts:
- removed C22: 1uF, Capacitor_SMD:C_0805_2012Metric, symbol Device:C_Small
- removed C23: 470nF, Capacitor_SMD:C_0805_2012Metric, symbol Device:C_Small
- removed J2: BattConn, Connector_PinSocket_2.54mm:PinSocket_1x03_P2.54mm_Vertical, symbol Connector_Generic:Conn_01x03
- removed R19: 10m 1%, Resistor_SMD:R_0805_2012Metric, symbol Device:R_Small_US
- removed R20, R21, R23: 5K1, Resistor_SMD:R_0805_2012Metric, symbol Device:R_Small_US
- removed R22: 1M8, Resistor_SMD:R_0805_2012Metric, symbol Device:R_Small_US
- removed U4: BQ27441-G1, Package_SON:Texas_S-PDSO-N12, symbol Battery_Management:BQ27441-G1
Connections:
- no-connect marks 1 -> 0
Other:
- note removed: "load or system voltage"
