File: realtime-communication/hardware/rt_hw_v1/rt_hw_v1.kicad_pcb (KiCad board)
At the start: 2 copper layers, 68 parts, among them J1 USB2UART, J6 ConnBattery, Q1 SS8050, Q2 SS8050, SW1 RST, SW3 Boot, SW4 5V_EN, SW9 PS Joystick, U1 74HCT245_TSSOP, U2 CH340C, U3 ESP32-S3-WROOM-1, U4 BQ27441-G1, U5 BQ24075RGT_DPPM, U6 TPS63002_SEPIC_5V, U7 ADS1115IDGS, U9 TPS63001_SEPIC_3V3

Commit message: add bq27441 single batt fuel gauge
Parts:
- added C22: 1uF, Capacitor_SMD:C_0805_2012Metric, F.Cu at (111.0, 84.8)
- added C23: 470nF, Capacitor_SMD:C_0805_2012Metric, F.Cu at (95.6, 83.0)
- added J2: BattConn, Connector_PinSocket_2.54mm:PinSocket_1x03_P2.54mm_Vertical, B.Cu at (99.1, 88.8)
- added R19: 10m 1%, Resistor_SMD:R_0805_2012Metric, F.Cu at (108.9, 84.8)
- added R20: 5K1, Resistor_SMD:R_0805_2012Metric, F.Cu at (101.4, 76.8)
- added R21: 5K1, Resistor_SMD:R_0805_2012Metric, F.Cu at (99.4, 76.8)
- added R22: 1M8, Resistor_SMD:R_0805_2012Metric, F.Cu at (110.9, 81.0)
- added R23: 5K1, Resistor_SMD:R_0805_2012Metric, F.Cu at (108.9, 81.0)
- moved U4 104.1 mm to (101.5, 83.0)
- moved C21 23.9 mm to (122.2, 89.0)
- moved R10 23.9 mm to (121.9, 79.0)
- moved R18 23.9 mm to (124.9, 79.8)
- moved R3 23.9 mm to (121.9, 81.2)
- moved U7 23.9 mm to (122.0, 85.8)
- moved BT1 3.21 mm to (162.5, 74.0)
Connections:
- SW9 pad 2: /AN1 -> /AIN0
- SW9 pad 5: /AN2 -> /AIN1
- U4 pad 1: unconnected-(U4-SDA-Pad1) -> /BQ27441_Batt_Fuel_Gauge/SDA
- U4 pad 10: unconnected-(U4-BIN-Pad10) -> /BQ27441_Batt_Fuel_Gauge/BIN
- U4 pad 12: unconnected-(U4-GPOUT-Pad12) -> /BQ27441_Batt_Fuel_Gauge/GPOUT
- U4 pad 13: unconnected-(U4-PAD-Pad13) -> GND
- U4 pad 2: unconnected-(U4-SCL-Pad2) -> /BQ27441_Batt_Fuel_Gauge/SCL
- U4 pad 3: unconnected-(U4-V_{SS}-Pad3) -> GND
- U4 pad 5: unconnected-(U4-V_{DD}-Pad5) -> Net-(U4-V_{DD})
- U4 pad 6: unconnected-(U4-BAT-Pad6) -> +BATT
- U4 pad 7: unconnected-(U4-SRN-Pad7) -> VSys
- U4 pad 8: unconnected-(U4-SRP-Pad8) -> +BATT
Routing:
- net +BATT: track 0.00 -> 37.2 mm, vias 0 -> 2
- net GND: track 8.93 -> 44.2 mm
- net +3.3V: track 18.8 -> 34.0 mm
- net /BQ27441_Batt_Fuel_Gauge/SDA: track 0.00 -> 14.1 mm
- net VSys: track 0.00 -> 11.3 mm
- net /BQ27441_Batt_Fuel_Gauge/GPOUT: track 0.00 -> 10.7 mm
- net /BQ27441_Batt_Fuel_Gauge/BIN: track 0.00 -> 10.5 mm
- net /BQ27441_Batt_Fuel_Gauge/SCL: track 0.00 -> 8.74 mm
- net Net-(U4-V_{DD}): track 0.00 -> 4.10 mm

Commit message: add regular sdcard to rt board
Parts:
- removed BT1: Battery_Cell, Battery:BatteryHolder_Bulgin_BX0034_1xAAA
- removed D32: red, LED_SMD:LED_0805_2012Metric_Pad1.15x1.40mm_HandSolder
- removed J6: ConnBattery, Connector_PinHeader_2.54mm:PinHeader_1x03_P2.54mm_Vertical
- removed SW4: 5V_EN, Button_Switch_SMD:SW_SPDT_PCM12
- removed U9: TPS63001_SEPIC_3V3, Package_SON:Texas_DRC0010J_ThermalVias
- added C24: 100nF, Capacitor_SMD:C_0805_2012Metric, F.Cu at (61.0, 94.9)
- added D6: red, LED_SMD:LED_0805_2012Metric_Pad1.15x1.40mm_HandSolder, F.Cu at (39.8, 27.4)
- added J3: ConnBattery, Connector_PinHeader_2.54mm:PinHeader_1x03_P2.54mm_Vertical, B.Cu at (24.0, 24.7)
- added J4: SD_Card_Receptacle, Connector_Card:SD_TE_2041021, F.Cu at (77.2, 97.2)
- added JP1: EN, Jumper:SolderJumper-3_P1.3mm_Open_RoundedPad1.0x1.5mm_NumberLabels, F.Cu at (95.3, 25.3)
- added JP2: EN, Jumper:SolderJumper-3_P1.3mm_Open_RoundedPad1.0x1.5mm_NumberLabels, F.Cu at (62.1, 61.9)
- added R24: 47K, Resistor_SMD:R_0805_2012Metric, F.Cu at (59.2, 109.4)
- added R25: 47K, Resistor_SMD:R_0805_2012Metric, F.Cu at (58.1, 106.5)
- added R26: 47K, Resistor_SMD:R_0805_2012Metric, F.Cu at (60.2, 106.5)
- added R27: 47K, Resistor_SMD:R_0805_2012Metric, F.Cu at (56.4, 91.2)
- added R28: 47K, Resistor_SMD:R_0805_2012Metric, F.Cu at (60.0, 91.2)
- added U8: TPS63002_SEPIC_5V, Package_SON:Texas_DRC0010J_ThermalVias, F.Cu at (61.8, 54.4)
- C10: value 1uF -> 10uF
- C4: value 4.7uF -> 1uF
- C6: value 10uF -> 4.7uF
- C7, C8: value 100nF -> 1uF
- R13: value 100 -> 1.13k
- R14: value 1.13k -> 1K5
- R17: value 1K5 -> 100
- R2, R32, R4: value 1k -> 10K
- R7: value 1.18k -> 2K2
- U6: value TPS63002_SEPIC_5V -> TPS63001
- moved C5 213.1 mm to (21.5, 28.7), turned to -90 degrees
- moved C4 207.3 mm to (26.5, 28.7), turned to -90 degrees
- moved C6 207.0 mm to (33.0, 22.7)
- moved R7 196.0 mm to (33.0, 18.2)
- moved U5 195.6 mm to (33.0, 28.9), turned to 90 degrees
- moved R13 195.4 mm to (33.0, 35.7)
- moved R6 194.4 mm to (33.0, 20.4)
- moved D4 194.2 mm to (37.5, 27.4), turned to -90 degrees
- moved R14 192.6 mm to (37.5, 31.4), turned to -90 degrees
- moved R15 191.1 mm to (39.8, 31.4), turned to -90 degrees
- moved L2 189.8 mm to (61.1, 43.4), turned to 180 degrees
- moved L1 180.4 mm to (76.8, 26.3), turned to -90 degrees
- moved C14 175.6 mm to (56.9, 58.4)
- moved C15 174.6 mm to (57.9, 61.4), turned to 90 degrees
- moved R17 173.5 mm to (55.8, 61.4), turned to -90 degrees
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Connections:
- net /BQ27441_Batt_Fuel_Gauge/BIN renamed /BIN
- C10 pad 1: VBUS -> VDD
- C11 pad 1: Net-(SW4-A) -> Net-(JP1-B)
- C12 pad 1: +5V -> +3.3V
- C13 pad 1: +5V -> +3.3V
- C15 pad 1: Net-(U9-EN) -> Net-(JP2-B)
- C16 pad 1: +3.3V -> +5V
- C17 pad 1: +3.3V -> +5V
- C4 pad 1: +BATT -> VBUS
- C5 pad 1: VDD -> +BATT
- R13 pad 1: VDD -> /ISET
- R13 pad 2: Net-(SW4-A) -> GND
- R14 pad 1: /ISET -> Net-(D4-A)
- R14 pad 2: GND -> VDD
- R15 pad 1: Net-(D4-A) -> Net-(D6-A)
- R16 pad 2: Net-(U9-EN) -> Net-(JP1-B)
- R17 pad 1: Net-(D32-A) -> VDD
- R17 pad 2: VDD -> Net-(JP2-B)
- R20 pad 2: /BQ27441_Batt_Fuel_Gauge/SDA -> /SDA
- R21 pad 2: /BQ27441_Batt_Fuel_Gauge/SCL -> /SCL
- R23 pad 2: /BQ27441_Batt_Fuel_Gauge/GPOUT -> /BQ27441_GPOUT
- R3 pad 2: /DRDY -> /ADS_DRDY
- U1 pad 2: /A0 -> /MOSI
- U3 pad 10: /IN1 -> /BQ27441_GPOUT
- U3 pad 12: /MAX31865DRDY -> /LED_CS
- U3 pad 17: /MAX31865CS -> /ADS_DRDY
- U3 pad 38: unconnected-(U3-IO2-Pad38) -> /SCL
- U3 pad 39: unconnected-(U3-IO1-Pad39) -> /SDA
- U4 pad 1: /BQ27441_Batt_Fuel_Gauge/SDA -> /SDA
- U4 pad 12: /BQ27441_Batt_Fuel_Gauge/GPOUT -> /BQ27441_GPOUT
- U4 pad 2: /BQ27441_Batt_Fuel_Gauge/SCL -> /SCL
- U5 pad 15: /SYSOFF -> GND
- U6 pad 1: +5V -> +3.3V
- U6 pad 10: +5V -> +3.3V
- U6 pad 7: Net-(SW4-A) -> Net-(JP1-B)
- U6 pad 8: Net-(SW4-A) -> Net-(JP1-B)
- U7 pad 2: /DRDY -> /ADS_DRDY
Routing:
- net /DAT1: track 0.00 -> 280.5 mm, vias 0 -> 5
- net VDD: track 0.00 -> 68.7 mm, vias 0 -> 2
- net GND: track 44.2 -> 109.3 mm
- net /TS: track 0.00 -> 30.0 mm
- net +5V: track 0.00 -> 25.0 mm
- net Net-(JP2-C): track 0.00 -> 21.8 mm
- net Net-(JP1-C): track 0.00 -> 21.8 mm
- net /TMR: track 0.00 -> 19.4 mm
- net /BQ27441_Batt_Fuel_Gauge/SDA: track 14.1 -> 0.00 mm
- net Net-(JP2-B): track 0.00 -> 13.8 mm
- net Net-(JP1-B): track 0.00 -> 13.8 mm
- net /ILIM: track 0.00 -> 12.0 mm
- net VSys: track 11.3 -> 0.00 mm
- net Net-(U6-L1): track 0.00 -> 10.8 mm
- net Net-(U8-L1): track 0.00 -> 10.8 mm
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
Commit message: finish routing rt hardware
Parts:
- C1, C2, C3, D1, D2, D3, SW9: moved to B.Cu
- U2: value CH340C -> CH340G
- moved R17 171.1 mm to (211.4, 132.5), turned to 0 degrees
- moved C15 168.4 mm to (211.4, 130.5), turned to 180 degrees
- moved C14 168.3 mm to (208.4, 131.5), turned to 90 degrees
- moved JP2 163.0 mm to (211.9, 126.2), turned to -90 degrees
- moved C4 160.4 mm to (162.7, 113.5)
- moved C5 160.4 mm to (157.7, 113.5)
- moved C6 160.4 mm to (169.2, 107.5)
- moved D4 160.4 mm to (173.7, 112.2)
- moved D6 160.4 mm to (175.9, 112.2)
- moved J3 160.4 mm to (160.2, 109.4)
- moved R13 160.4 mm to (169.2, 120.5)
- moved R14 160.4 mm to (173.7, 116.2)
- moved R15 160.4 mm to (175.9, 116.2)
- moved R6 160.4 mm to (169.2, 105.2)
- moved R7 160.4 mm to (169.2, 103.0)
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Connections:
- R19 pad 1: VSys -> VDD
- SW9 pad 2: /AIN0 -> /AIN1
- SW9 pad 5: /AIN1 -> /AIN0
- U3 pad 11: /IN2 -> /CARD_DETECT
- U3 pad 13: /IN3 -> unconnected-(U3-IO19-Pad13)
- U3 pad 14: /IN4 -> unconnected-(U3-IO20-Pad14)
- U3 pad 22: /RESET -> /DAT3
- U3 pad 23: /IN5 -> /ANSW
- U3 pad 5: unconnected-(U3-IO5-Pad5) -> /DAT0
- U3 pad 6: unconnected-(U3-IO6-Pad6) -> /DAT1
- U3 pad 7: unconnected-(U3-IO7-Pad7) -> /DAT2
- U3 pad 8: /DC -> /CLK
- U3 pad 9: /BLK -> /CMD
- U4 pad 7: VSys -> VDD
Routing:
- net GND: track 109.3 -> 645.5 mm, vias 0 -> 7
- net +3.3V: track 43.8 -> 441.8 mm, vias 0 -> 7
- net /DAT1: track 280.5 -> 57.7 mm, vias 5 -> 2
- net /SCL: track 8.48 -> 220.1 mm, vias 0 -> 3
- net /SDA: track 6.54 -> 182.1 mm, vias 0 -> 3
- net VDD: track 68.7 -> 205.2 mm, vias 2 -> 5
- net VBUS: track 5.29 -> 115.3 mm, vias 0 -> 2
- net /LED_CS: track 0.00 -> 107.5 mm, vias 0 -> 2
- net /EN: track 0.00 -> 98.6 mm, vias 0 -> 2
- net /IO0: track 0.00 -> 98.5 mm, vias 0 -> 2
- net +5V: track 25.0 -> 122.9 mm, vias 0 -> 1
- net +BATT: track 29.3 -> 116.1 mm, vias 2 -> 4
- net /CMD: track 0.00 -> 73.4 mm, vias 0 -> 2
- net /ANSW: track 0.00 -> 65.8 mm, vias 0 -> 2
- net /CLK: track 0.00 -> 65.0 mm, vias 0 -> 2
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Other:
- board outline added: 113.4 x 86.2 mm
- board text added: "Routed at 19:41 24 September 2026"
