File: realtime-communication/hardware/rt_hw_v1/rt_hw_v1.kicad_pcb (KiCad board)
At the start: 2 copper layers, 113.4 x 86.2 mm, 83 parts, among them J1 USB2UART, J2 BattConn, J3 ConnBattery, J4 SD_Card_Receptacle, Q1 SS8050, Q2 SS8050, SW1 RST, SW3 Boot, SW9 PS Joystick, U1 74HCT245_TSSOP, U2 CH340G, U3 ESP32-S3-WROOM-1, U4 BQ27441-G1, U5 BQ24075RGT_DPPM, U6 TPS63001, U7 ADS1115IDGS, U8 TPS63002_SEPIC_5V

Commit message: add rt-hw-v1 diy fabrication files
Parts:
- moved J1 25.9 mm to (213.1, 84.0)
- moved R8 21.8 mm to (210.7, 94.6)
- moved R5 21.4 mm to (215.8, 94.5)
Routing:
- net Net-(U2-UD+): track 27.6 -> 52.3 mm, vias 0 -> 2
- net VBUS: track 115.3 -> 92.3 mm
- net Net-(U2-UD-): track 26.2 -> 44.1 mm, vias 0 -> 2
- net Net-(J1-CC1): track 13.0 -> 7.13 mm
- net Net-(J1-CC2): track 12.7 -> 7.11 mm
- net +3.3V: track 441.8 -> 444.0 mm
- net GND: track 645.5 -> 647.3 mm
- net /RXD0: track 43.0 -> 41.8 mm
Other:
- board size 113.4 x 86.2 mm -> 113.4 x 65 mm
- board text removed: "Routed at 19:41 24 September 2026"
