File: realtime-communication/hardware/rt_hw_v1/rt_hw_v1.kicad_sch (KiCad schematic)
At the start: 67 parts, among them J1 USB2UART, J6 ConnBattery, Q1 SS8050, Q2 SS8050, SW1 RST, SW3 Boot, SW4 5V_EN, SW9 PS Joystick, U1 74HCT245_TSSOP, U2 CH340C, U3 ESP32-S3-WROOM-1, U5 BQ24075RGT_DPPM, U6 TPS63002_SEPIC_5V, U7 ADS1115IDGS, U9 TPS63001_SEPIC_3V3

Commit message: add regular sdcard to rt board
Parts:
- removed BT1: Battery_Cell, Battery:BatteryHolder_Bulgin_BX0034_1xAAA, symbol Device:Battery_Cell
- removed D32: red, LED_SMD:LED_0805_2012Metric_Pad1.15x1.40mm_HandSolder, symbol Device:LED
- removed J6: ConnBattery, Connector_PinHeader_2.54mm:PinHeader_1x03_P2.54mm_Vertical, symbol Connector_Generic:Conn_01x03
- removed SW4: 5V_EN, Button_Switch_SMD:SW_SPDT_PCM12, symbol Switch:SW_Push_SPDT
- removed U6: TPS63002_SEPIC_5V, Package_SON:Texas_DRC0010J_ThermalVias, symbol Regulator_Switching:TPS63002
- removed U9: TPS63001_SEPIC_3V3, Package_SON:Texas_DRC0010J_ThermalVias, symbol Regulator_Switching:TPS63001
- added C22: 1uF, Capacitor_SMD:C_0805_2012Metric, symbol Device:C_Small
- added C23: 470nF, Capacitor_SMD:C_0805_2012Metric, symbol Device:C_Small
- added C24: 100nF, Capacitor_SMD:C_0805_2012Metric, symbol Device:C_Small
- added D6: red, LED_SMD:LED_0805_2012Metric_Pad1.15x1.40mm_HandSolder, symbol Device:LED
- added J2: BattConn, Connector_PinSocket_2.54mm:PinSocket_1x03_P2.54mm_Vertical, symbol Connector_Generic:Conn_01x03
- added J3: ConnBattery, Connector_PinHeader_2.54mm:PinHeader_1x03_P2.54mm_Vertical, symbol Connector_Generic:Conn_01x03
- added J4: SD_Card_Receptacle, Connector_Card:SD_TE_2041021, symbol Connector:SD_Card_Receptacle
- added JP1, JP2: EN, Jumper:SolderJumper-3_P1.3mm_Open_RoundedPad1.0x1.5mm_NumberLabels, symbol Jumper:SolderJumper_3_Open
- added R19: 10m 1%, Resistor_SMD:R_0805_2012Metric, symbol Device:R_Small_US
- added R20, R21, R23: 5K1, Resistor_SMD:R_0805_2012Metric, symbol Device:R_Small_US
- added R22: 1M8, Resistor_SMD:R_0805_2012Metric, symbol Device:R_Small_US
- added R24, R25, R26, R27, R28: 47K, Resistor_SMD:R_0805_2012Metric, symbol Device:R_Small_US
- added U4: BQ27441-G1, Package_SON:Texas_S-PDSO-N12, symbol Battery_Management:BQ27441-G1
- added U6: TPS63001, Package_SON:Texas_DRC0010J_ThermalVias, symbol Regulator_Switching:TPS63001
- added U8: TPS63002_SEPIC_5V, Package_SON:Texas_DRC0010J_ThermalVias, symbol Regulator_Switching:TPS63002
- C10: value 1uF -> 10uF
- C4: value 4.7uF -> 1uF
- C6: value 10uF -> 4.7uF
- C7, C8: value 100nF -> 1uF
- R13: value 100 -> 1.13k
- R14: value 1.13k -> 1K5
- R17: value 1K5 -> 100
- R2, R32, R4: value 1k -> 10K
- R7: value 1.18k -> 2K2
Connections:
- net A0 is gone; now on net MOSI: U1.2 (A0)
- net MAX31865CS is gone; now on net ADS_DRDY: U3.17 (IO9)
- net MAX31865DRDY is gone; now on net LED_CS: U3.12 (IO8)
- net SYSOFF is gone; now on net GND: U5.15 (SYSOFF)
- net +3.3V: now also C12.1, C13.1, C24.1, J4.4 (VDD), R20.1, R21.1, R22.1, R23.1, R24.1, R25.1, R26.1, R27.1, R28.1, U6.1 (VOUT), U6.10 (FB); no longer C16.1, C17.1
- net +5V: now also C16.1, C17.1, U8.1 (VOUT), U8.10 (FB); no longer C12.1, C13.1
- net +BATT: now also C5.1, C22.1, J2.1 (Pin_1), J3.1 (Pin_1), R19.2, U4.6 (BAT), U4.8 (SRP); no longer C4.1
- net GND: now also R13.2, C22.2, C23.2, C24.2, J2.3 (Pin_3), J3.3 (Pin_3), J4.3 (VSS), J4.6 (VSS), JP1.1 (A), JP2.1 (A), U4.13 (PAD), U4.3 (V_{SS}), U6.11 (PGND), U6.3 (PGND), U6.9 (GND), U8.11 (PGND), U8.3 (PGND), U8.9 (GND); no longer R14.2
- net ISET: now also R13.1; no longer R14.1
- net SCL: now also U3.38 (IO2), R21.2, U4.2 (SCL)
- net SDA: now also U3.39 (IO1), R20.2, U4.1 (SDA)
- net TS: now also J3.2 (Pin_2)
- net VBUS: now also C4.1; no longer C10.1
- net VDD: now also C10.1, R14.2, R17.1, U6.5 (VIN), U8.5 (VIN); no longer C5.1, R13.1, R17.2
- net ~{CHG}: now also D6.1 (K)
- net at C15.1: now also R17.2, JP2.3 (B), U8.7 (PS/SYNC), U8.8 (VINA); no longer R16.2
- net at R15.1: now also D6.2 (A); no longer D4.2 (A)
- net at L2.1: now also U8.2 (L2)
- net at L2.2: now also U8.4 (L1)
- net at C11.1: now also R16.2, JP1.3 (B), U6.7 (PS/SYNC), U6.8 (VINA); no longer R13.2
- net at L1.1: now also U6.2 (L2)
- net at L1.2: now also U6.4 (L1)
- net DRDY renamed ADS_DRDY
- net IN1 renamed BQ27441_GPOUT
- net BQ27441_GPOUT: now also R23.2, U4.12 (GPOUT)
- new net: JP1.2 (C), U6.6 (EN)
- new net: C23.1, U4.5 (V_{DD})
- new net: D4.2 (A), R14.1
- new net: JP2.2 (C), U8.6 (EN)
- new net BIN: R22.2, U4.10 (BIN)
- new net CARD_DETECT: J4.10 (CARD_DETECT), R24.2
- new net CLK: J4.5 (CLK)
- new net CMD: J4.2 (CMD)
- new net DAT0: J4.7 (DAT0), R25.2
- new net DAT1: J4.8 (DAT1), R26.2
- new net DAT2: J4.9 (DAT2), R27.2
- new net DAT3: J4.1 (CD/DAT3), R28.2
- new net VSys: R19.1, U4.7 (SRN)
Other:
- removed sheet BQ27441_Batt_Fuel_Gauge
- note added: "Description"
- note added: "Input, May Come From USB"
- note added: "Min 1.8V - Max 5.5V"
- note added: "Output, managed voltage, value is between VBUS, or VBAT"
- note added: "SEPIC 3V3"
- note added: "TS is thermistor for temp sensor"
- note added: "let sdmmc = Sdmmc::new_4bit( p.SDIO, p.DMA2_CH3, Irqs, p.PC12, p.PD2, p.PC8, p.PC9, p.PC10, p.PC11, Default::default(), );"
- note added: "load or system voltage"
- note removed: "Program the Input Current Limit (ILIM) RILIM = KILIM / II_MAX KILIM = 1550 AΩ from the electrical characteristics table. RISET = 1550 AΩ / 1.3 A = 1.192 kΩ -> 1.18 kΩ"
- note removed: "SEPIC 3.3V"
- title: (none) -> Real Time Block Dev Board V0.0.1

Commit message: finish routing rt hardware
Parts:
- U2: value CH340C -> CH340G
Connections:
- net BLK is gone; now on net CMD: U3.9 (IO16)
- net DC is gone; now on net CLK: U3.8 (IO15)
- net IN2 is gone; now on net CARD_DETECT: U3.11 (IO18)
- net IN5 is gone; now on net ANSW: U3.23 (IO21)
- net RESET is gone; now on net DAT3: U3.22 (IO14)
- net VSys is gone; now on net VDD: R19.1, U4.7 (SRN)
- net AIN0: now also SW9.5 (DTA); no longer SW9.2 (DTA)
- net AIN1: now also SW9.2 (DTA); no longer SW9.5 (DTA)
- net DAT0: now also U3.5 (IO5)
- net DAT1: now also U3.6 (IO6)
- net DAT2: now also U3.7 (IO7)
- net IN3: no longer names the net of U3.13 (IO19)
- net IN4: no longer names the net of U3.14 (IO20)
Other:
- moved on the sheet: C1, C10, C11, C12, C13, C14, C15, C16, C17, C18, C19, C2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
