File: ph_module/ph_module.kicad_sch (KiCad schematic)
At the start: 0 parts

Commit message: some update
Parts:
- added U1: LMV324, Package_SO:SOIC-14_3.9x8.7mm_P1.27mm, symbol Amplifier_Operational:LMV324
- added U2: LMC7660, Package_SO:SOIC-8_3.9x4.9mm_P1.27mm, symbol Regulator_SwitchedCapacitor:LMC7660
