File: tds_module/tds_module.kicad_sch (KiCad schematic)
At the start: 0 parts

Commit message: some update
Parts:
- added U1: AMS1117-3.3, Package_TO_SOT_SMD:SOT-223-3_TabPin2, symbol Regulator_Linear:AMS1117-3.3
- added U2: LMC7660, symbol Regulator_SwitchedCapacitor:LMC7660
- added U3: 74HC4060, Package_SO:SOIC-16_3.9x9.9mm_P1.27mm, symbol 74xx:74HC4060
- added U4: LMV324, Package_SO:SOIC-14_3.9x8.7mm_P1.27mm, symbol Amplifier_Operational:LMV324
Other:
- note added: "based on the docs, freq cd4060 is around 45.5Khz then it divided by 2^5 (because it q4) then final result is 45.5Khz/32 = 1.4Khz the "pulse" generator is used to create -0.2v to 0.2v it used to "electrochemical measurement""
