File: mosokik/mosokik.kicad_sch (KiCad schematic)
At the start: 0 parts

Commit message: start to create schematic and board in mosokik
Parts:
- added C10: 22uF, Capacitor_SMD:C_0805_2012Metric_Pad1.18x1.45mm_HandSolder, symbol Device:C
- added C11, C13, C16, C17: 10uF, Capacitor_SMD:C_0805_2012Metric_Pad1.18x1.45mm_HandSolder, symbol Device:C
- added C14: 0.1uF, Capacitor_SMD:C_0805_2012Metric_Pad1.18x1.45mm_HandSolder, symbol Device:C
- added C15: 1uF, Capacitor_SMD:C_0805_2012Metric_Pad1.18x1.45mm_HandSolder, symbol Device:C
- added C2, C4, C7, C8: 100nF, Capacitor_SMD:C_0805_2012Metric_Pad1.18x1.45mm_HandSolder, symbol Device:C
- added C22, C23: 4.7uF, Capacitor_SMD:C_0805_2012Metric_Pad1.18x1.45mm_HandSolder, symbol Device:C
- added C3: 100nF, Capacitor_SMD:C_0805_2012Metric, symbol Device:C_Small
- added Card1: TF PUSH, easyeda2kicad:TF-SMD_TF-PUSH, symbol easyeda2kicad:TFPUSH
- added D4: VDD, LED_SMD:LED_1206_3216Metric_Pad1.42x1.75mm_HandSolder, symbol Device:LED
- added D5: green, LED_SMD:LED_0805_2012Metric_Pad1.15x1.40mm_HandSolder, symbol Device:LED
- added D6: red, LED_SMD:LED_0805_2012Metric_Pad1.15x1.40mm_HandSolder, symbol Device:LED
- added H1, H2, H3, H4: MountingHole_Pad, MountingHole:MountingHole_3.5mm_Pad, symbol Mechanical:MountingHole_Pad
- added J1: USB2UART, Connector_USB:USB_C_Receptacle_GCT_USB4110, symbol Connector:USB_C_Receptacle_USB2.0_14P
- added J2: 1.47 IPS LCD, Connector_PinHeader_2.54mm:PinHeader_1x08_P2.54mm_Vertical, symbol Connector_Generic:Conn_01x08
- added J3: ConnBattery, Connector_PinHeader_2.54mm:PinHeader_1x03_P2.54mm_Vertical, symbol Connector_Generic:Conn_01x03
- added J4, J7: LCD CONN BUFF, Connector_PinHeader_2.54mm:PinHeader_1x08_P2.54mm_Vertical, symbol Connector_Generic:Conn_01x08
- added J5: TOP_CONN, Connector_PinHeader_2.54mm:PinHeader_2x10_P2.54mm_Vertical, symbol Connector_Generic:Conn_02x10_Odd_Even
- added L1: 22uH 1A, Inductor_SMD:L_Bourns_SRP7028A_7.3x6.6mm, symbol Device:L
- added Q1, Q2: SS8050, Package_TO_SOT_SMD:SOT-23_Handsoldering, symbol Transistor_BJT:BC817
- added R10, R25, R26, R27, R9: 47K, Resistor_SMD:R_0805_2012Metric, symbol Device:R_Small_US
- added R11, R12: 10k, Resistor_SMD:R_0805_2012Metric_Pad1.20x1.40mm_HandSolder, symbol Device:R_US
- added R13: 1k, Resistor_SMD:R_0805_2012Metric_Pad1.20x1.40mm_HandSolder, symbol Device:R_US
- added R15: 100, Resistor_SMD:R_0805_2012Metric_Pad1.20x1.40mm_HandSolder, symbol Device:R_US
- added R16: 46.4K, Resistor_SMD:R_0805_2012Metric_Pad1.20x1.40mm_HandSolder, symbol Device:R_US
- added R17: 2K2, Resistor_SMD:R_0805_2012Metric_Pad1.20x1.40mm_HandSolder, symbol Device:R_US
- added R18: 1.13k, Resistor_SMD:R_0805_2012Metric_Pad1.20x1.40mm_HandSolder, symbol Device:R_US
- added R19, R22: 10K, Resistor_SMD:R_0805_2012Metric_Pad1.20x1.40mm_HandSolder, symbol Device:R_US
- added R20, R21: 1K5, Resistor_SMD:R_0805_2012Metric_Pad1.20x1.40mm_HandSolder, symbol Device:R_US
- added R23, R24: 4K7, Resistor_SMD:R_0805_2012Metric_Pad1.20x1.40mm_HandSolder, symbol Device:R_US
- added R5, R6: 5K1, Resistor_SMD:R_0805_2012Metric_Pad1.20x1.40mm_HandSolder, symbol Device:R_US
- added SW1: RST, Button_Switch_SMD:SW_SPST_PTS810, symbol Switch:SW_Push
- added SW3: Boot, Button_Switch_SMD:SW_SPST_PTS810, symbol Switch:SW_Push
- added U1: CH340C, Package_SO:SOIC-16_3.9x9.9mm_P1.27mm, symbol Interface_USB:CH340C
- added U2: ESP32-S3-WROOM-1, RF_Module:ESP32-S3-WROOM-1, symbol RF_Module:ESP32-S3-WROOM-1
- added U4: TPS63001_SEPIC_3V3, Package_SON:Texas_DRC0010J_ThermalVias, symbol Regulator_Switching:TPS63001
- added U5: BQ24075RGT_DPPM, Package_DFN_QFN:VQFN-16-1EP_3x3mm_P0.5mm_EP1.6x1.6mm, symbol Battery_Management:BQ24075RGT
- added U7: MAX17048G+T10, easyeda2kicad:TDFN-8_L2.0-W2.0-P0.50-BL-EP1.2, symbol easyeda2kicad:MAX17048G+T10
Connections:
- new net: D5.2 (A), R20.1
- new net: J4.1 (Pin_1), J7.1 (Pin_1)
- new net: J4.2 (Pin_2), J7.2 (Pin_2)
- new net: J4.3 (Pin_3), J7.3 (Pin_3)
- new net: J4.4 (Pin_4), J7.4 (Pin_4)
- new net: J4.5 (Pin_5), J7.5 (Pin_5)
- new net: J4.6 (Pin_6), J7.6 (Pin_6)
- new net: J4.7 (Pin_7), J7.7 (Pin_7)
- new net: J4.8 (Pin_8), J7.8 (Pin_8)
- new net: D4.2 (A), R13.2
- new net: Q1.1 (B), R11.1
- new net: C14.1, R15.2, U4.6 (EN), U4.7 (PS/SYNC), U4.8 (VINA)
- new net: J1.A6 (D+), J1.B6 (D+), U1.5 (UD+)
- new net: J1.A7 (D-), J1.B7 (D-), U1.6 (UD-)
- new net: D6.2 (A), R21.1
- new net: L1.1, U4.2 (L2)
- new net: L1.2, U4.4 (L1)
- new net: Q2.1 (B), R12.1
- new net: J1.A5 (CC1), R5.2
- new net: J1.B5 (CC2), R6.2
- new net +3.3V: C10.1, C11.1, C16.1, C17.1, C3.1, C7.1, C8.1, Card1.4 (VDD), J2.2 (Pin_2), J5.4 (Pin_4), R10.1, R19.1, R20.2, R21.2, R22.1, R23.1, R24.1, R25.1, R26.1, R27.1, R9.1, U1.16 (VCC), U1.4 (V3), U2.2 (3V3), U4.1 (VOUT), U4.10 (FB)
- new net +BATT: C22.1, J3.1 (Pin_1), J5.6 (Pin_6), U5.2 (BAT), U5.3 (BAT), U7.2 (CELL), U7.3 (VDD)
- new net BLK: J2.8 (Pin_8), U2.9 (IO16)
- new net CARD_DETECT: Card1.CD, R27.2
- new net CLK: Card1.5 (CLX), U2.17 (IO9)
- new net CMD: Card1.3 (CMD), U2.12 (IO8)
- new net CS: J2.7 (Pin_7), U2.18 (IO10)
- new net DAT0: Card1.7 (DAT0), R25.2, U2.4 (IO4)
- new net DAT1: Card1.8 (DAT1), R26.2, U2.5 (IO5)
- new net DAT2: Card1.1 (DAT2), R9.2, U2.6 (IO6)
- new net DAT3: Card1.2 (CD/DAT3), R10.2, U2.7 (IO7)
- new net DC: J2.6 (Pin_6), U2.8 (IO15)
- new net DTR: Q2.2 (E), R11.2, U1.13 (~{DTR})
- new net EN: C2.1, Q1.3 (C), R19.2, SW1.2, U2.3 (EN)
- new net GND: C10.2, C11.2, C13.2, C14.2, C15.2, C16.2, C17.2, C2.2, C22.2, C23.2, C3.2, C4.2, C7.2, C8.2, Card1.6 (VSS), D4.1 (K), J1.A1 (GND), J1.A12 (GND), J1.B1 (GND), J1.B12 (GND), J2.1 (Pin_1), J3.3 (Pin_3), J5.8 (Pin_8), R16.2, R17.2, R18.2, R5.1, R6.1, SW1.1, SW3.1, U1.1 (GND), U2.1 (GND), U2.40 (GND), U2.41 (GND), U4.11 (PGND), U4.3 (PGND), U4.9 (GND), U5.15 (SYSOFF), U5.17 (VSS), U5.4 (~{CE}), U5.6 (EN1), U5.8 (VSS), U7.1 (CTG), U7.4 (GND), U7.6 (QSTRT), U7.9 (EP)
- new net ILIM: R17.1, U5.12 (ILIM)
- new net IO0: C4.1, Q2.3 (C), SW3.2, U2.27 (IO0)
- new net IO17: J5.1 (Pin_1), U2.10 (IO17)
- new net IO18: J5.3 (Pin_3), U2.11 (IO18)
- new net IO19: J5.5 (Pin_5), U2.13 (IO19)
- new net IO20: J5.7 (Pin_7), U2.14 (IO20)
- new net IO21: J5.9 (Pin_9), U2.23 (IO21)
- new net IO41: J5.11 (Pin_11), U2.34 (IO41)
- new net IO42: J5.13 (Pin_13), U2.35 (IO42)
- new net IO45: J5.15 (Pin_15), U2.26 (IO45)
- new net IO46: J5.17 (Pin_17), U2.16 (IO46)
- new net IO47: J5.19 (Pin_19), U2.24 (IO47)
- new net IO48: J5.10 (Pin_10), U2.25 (IO48)
- new net ISET: R18.1, U5.16 (ISET)
- new net MISO: J5.20 (Pin_20), U2.21 (IO13)
- new net MOSI: J2.4 (Pin_4), J5.16 (Pin_16), U2.19 (IO11)
- new net RESET: J2.5 (Pin_5), U2.22 (IO14)
- new net RTS: Q1.2 (E), R12.2, U1.14 (~{RTS})
- new net RXD0: U1.2 (TXD), U2.36 (RXD0)
- new net SCK: J2.3 (Pin_3), J5.18 (Pin_18), U2.20 (IO12)
- new net SCL: J5.14 (Pin_14), R24.2, U2.38 (IO2), U7.7 (SCL)
- new net SDA: J5.12 (Pin_12), R23.2, U2.39 (IO1), U7.8 (SDA)
- new net TMR: R16.1, U5.14 (TMR)
- new net TS: J3.2 (Pin_2), U5.1 (TS)
- new net TXD0: U1.3 (RXD), U2.37 (TXD0)
- new net VBUS: C15.1, J1.A4 (VBUS), J1.A9 (VBUS), J1.B4 (VBUS), J1.B9 (VBUS), J5.2 (Pin_2), U5.13 (IN)
- new net VDD: C13.1, C23.1, R13.1, R15.1, U4.5 (VIN), U5.10 (OUT), U5.11 (OUT), U5.5 (EN2)
- new net ~{ALRT}: R22.2, U2.31 (IO38), U7.5 (~{ALRT})
- new net ~{CHG}: D6.1 (K), U2.33 (IO40), U5.9 (~{CHG})
- new net ~{PGOOD}: D5.1 (K), U2.32 (IO39), U5.7 (~{PGOOD})
- no-connect marks 0 -> 19
Other:
- note added: "DPPM"
- note added: "ESP32-S3-WROOM-1"
- note added: "GND VCC SCL SDA RES DC CS BLK"
- note added: "Program Fast-Charge Safety Timer (TMR): RTMR = tMAXCHG / (10 × KTMR ) KTMR = 48 s/kΩ from the electrical characteristics table. RTMR = (6.25 hr × 3600 s/hr) / (10 × 48 s/kΩ) = 46.8 kΩ -> 46.4 kΩ"
- note added: "Program the Fast Charge Current (ISET): RISET = KISET / ICHG KISET = 890 AΩ from the electrical characteristics table. RISET = 890 AΩ / 0.8 A = 1.1125 kΩ -> 1.13 kΩ"
- note added: "SEPIC 3.3V"
- note added: "dynamic power path management"
- note added: "let sdmmc = Sdmmc::new_4bit( p.SDIO, p.DMA2_CH3, Irqs, p.PC12, p.PD2, p.PC8, p.PC9, p.PC10, p.PC11, Default::default(), );"
- note added: "miso - Also known as q, this is the input of the serial stream into the ESP32 mosi - Also known as d, this is the output of the serial stream from the ESP32 sclk - Clock signal. Each data bit is clocked out or in on the positive or negative edge of this signal quadwp - Write Protect signal. Only used for 4-bit (qio/qout) transactions. quadhd - Hold signal. Only used for 4-bit (qio/qout) transacti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"
- title: (none) -> Mosokik

Commit message: lazy route update
Parts:
- removed H1, H2, H3, H4: MountingHole_Pad, MountingHole:MountingHole_3.5mm_Pad, symbol Mechanical:MountingHole_Pad
- J5: footprint Connector_PinHeader_2.54mm:PinHeader_2x10_P2.54mm_Vertical -> Connector_PinHeader_2.54mm:PinHeader_2x10_P2.54mm_Horizontal
Connections:
- no-connect marks 19 -> 15

Commit message: unrouted 8 pieces
Connections:
- net +3.3V: now also J5.16 (Pin_16); no longer J5.4 (Pin_4)
- net +BATT: now also J5.18 (Pin_18); no longer J5.6 (Pin_6)
- net GND: now also J5.20 (Pin_20); no longer J5.8 (Pin_8)
- net IO17: now also J5.19 (Pin_19); no longer J5.1 (Pin_1)
- net IO18: now also J5.17 (Pin_17); no longer J5.3 (Pin_3)
- net IO19: now also J5.15 (Pin_15); no longer J5.5 (Pin_5)
- net IO20: now also J5.13 (Pin_13); no longer J5.7 (Pin_7)
- net IO21: now also J5.3 (Pin_3); no longer J5.9 (Pin_9)
- net IO41: now also J5.6 (Pin_6); no longer J5.11 (Pin_11)
- net IO42: now also J5.8 (Pin_8); no longer J5.13 (Pin_13)
- net IO45: now also J5.4 (Pin_4); no longer J5.15 (Pin_15)
- net IO46: now also J5.11 (Pin_11); no longer J5.17 (Pin_17)
- net IO47: now also J5.1 (Pin_1); no longer J5.19 (Pin_19)
- net IO48: now also J5.2 (Pin_2); no longer J5.10 (Pin_10)
- net MISO: now also J5.5 (Pin_5); no longer J5.20 (Pin_20)
- net MOSI: now also J5.9 (Pin_9); no longer J5.16 (Pin_16)
- net SCK: now also J5.7 (Pin_7); no longer J5.18 (Pin_18)
- net SCL: now also J5.10 (Pin_10); no longer J5.14 (Pin_14)
- net VBUS: now also J5.14 (Pin_14); no longer J5.2 (Pin_2)
