File: mosokik/mosokik.kicad_pcb (KiCad board)
At the start: 2 copper layers, 60 x 60 mm, 58 parts, among them J1 USB2UART, J2 1.47 IPS LCD, J3 ConnBattery, J4 LCD CONN BUFF, J5 TOP_CONN, J7 LCD CONN BUFF, Q1 SS8050, Q2 SS8050, SW1 RST, SW3 Boot, U1 CH340C, U2 ESP32-S3-WROOM-1, U4 TPS63001_SEPIC_3V3, U5 BQ24075RGT_DPPM, U7 MAX17048G+T10

Commit message: lazy route update
Parts:
- removed H1, H2, H3, H4: MountingHole_Pad, MountingHole:MountingHole_3.5mm_Pad
- J5: footprint Connector_PinHeader_2.54mm:PinHeader_2x10_P2.54mm_Vertical -> Connector_PinHeader_2.54mm:PinHeader_2x10_P2.54mm_Horizontal; moved to F.Cu
- moved C16 100.8 mm to (152.5, 105.4)
- moved C14 96.0 mm to (158.5, 111.3), turned to 90 degrees
- moved R15 94.6 mm to (160.6, 111.3), turned to 90 degrees
- moved D4 94.5 mm to (152.4, 118.6)
- moved C7 94.1 mm to (153.4, 85.7), turned to 180 degrees
- moved R6 94.0 mm to (152.5, 82.6), turned to 90 degrees
- moved R5 91.2 mm to (154.6, 82.6), turned to 90 degrees
- moved C17 90.2 mm to (152.5, 103.2)
- moved L1 86.0 mm to (140.3, 111.7), turned to -90 degrees
- moved C13 84.5 mm to (145.6, 111.9), turned to 90 degrees
- moved R13 83.2 mm to (152.5, 116.4)
- moved R12 79.4 mm to (158.0, 103.7), turned to 90 degrees
- moved R11 77.6 mm to (164.2, 103.7), turned to -90 degrees
- moved R22 77.0 mm to (126.1, 91.3)
- moved U7 76.3 mm to (126.1, 89.0), turned to -90 degrees
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Routing:
- net GND: track 0.00 -> 138.4 mm, vias 0 -> 1
- net VDD: track 0.00 -> 89.7 mm, vias 0 -> 2
- net +3.3V: track 0.00 -> 61.1 mm, vias 0 -> 1
- net /~{PGOOD}: track 0.00 -> 47.0 mm
- net /~{CHG}: track 0.00 -> 46.6 mm, vias 0 -> 2
- net +BATT: track 0.00 -> 40.3 mm, vias 0 -> 1
- net /IO0: track 0.00 -> 32.6 mm, vias 0 -> 2
- net /TXD0: track 0.00 -> 31.3 mm
- net /IO41: track 0.00 -> 29.8 mm, vias 0 -> 1
- net /DTR: track 0.00 -> 27.7 mm
- net /TS: track 0.00 -> 26.8 mm, vias 0 -> 1
- net /RXD0: track 0.00 -> 25.9 mm
- net /~{ALRT}: track 0.00 -> 21.8 mm, vias 0 -> 1
- net /EN: track 0.00 -> 19.9 mm, vias 0 -> 2
- net /DAT1: track 0.00 -> 17.9 mm, vias 0 -> 1
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
Commit message: need re-do on component placement
Routing:
- net +3.3V: track 61.1 -> 332.3 mm, vias 1 -> 10
- net /DAT1: track 17.9 -> 167.5 mm, vias 1 -> 7
- net /SCK: track 3.85 -> 152.1 mm, vias 1 -> 3
- net GND: track 138.4 -> 260.2 mm, vias 1 -> 7
- net /BLK: track 8.94 -> 108.7 mm
- net /~{ALRT}: track 21.8 -> 106.4 mm, vias 1 -> 2
- net /IO46: track 7.52 -> 91.2 mm, vias 1 -> 3
- net /CMD: track 5.16 -> 85.0 mm, vias 1 -> 2
- net /IO19: track 8.33 -> 86.1 mm
- net VBUS: track 15.8 -> 91.6 mm, vias 0 -> 2
- net /CLK: track 4.78 -> 75.6 mm, vias 1 -> 2
- net /EN: track 19.9 -> 86.0 mm, vias 2 -> 3
- net /IO21: track 7.45 -> 53.6 mm, vias 1 -> 2
- net /DAT2: track 13.1 -> 55.3 mm, vias 1 -> 2
- net /MISO: track 6.80 -> 41.5 mm
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
Commit message: unrouted 8 pieces
Parts:
- moved SW1 52.3 mm to (171.1, 81.2), turned to 180 degrees
- moved SW3 52.1 mm to (171.1, 85.3), turned to 180 degrees
- moved C2 46.5 mm to (167.0, 81.2), turned to -90 degrees
- moved C4 46.3 mm to (166.9, 85.3), turned to -90 degrees
- moved Card1 42.9 mm to (129.5, 101.0), turned to -90 degrees
- moved R19 41.9 mm to (164.6, 83.3), turned to 90 degrees
- moved R9 33.6 mm to (139.8, 107.7), turned to 180 degrees
- moved R10 30.4 mm to (139.8, 105.7), turned to 180 degrees
- moved L1 28.9 mm to (166.9, 123.1)
- moved R22 28.1 mm to (140.7, 115.3)
- moved U7 28.1 mm to (140.7, 113.0)
- moved R25 25.5 mm to (139.8, 100.7), turned to 180 degrees
- moved C15 24.4 mm to (134.1, 124.0)
- moved D4 24.0 mm to (175.1, 126.5)
- moved R13 24.0 mm to (175.2, 124.3)
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Connections:
- J5 pad 1: /IO17 -> /IO47
- J5 pad 10: /IO48 -> /SCL
- J5 pad 11: /IO41 -> /IO46
- J5 pad 13: /IO42 -> /IO20
- J5 pad 14: /SCL -> VBUS
- J5 pad 15: /IO45 -> /IO19
- J5 pad 16: /MOSI -> +3.3V
- J5 pad 17: /IO46 -> /IO18
- J5 pad 18: /SCK -> +BATT
- J5 pad 19: /IO47 -> /IO17
- J5 pad 2: VBUS -> /IO48
- J5 pad 20: /MISO -> GND
- J5 pad 3: /IO18 -> /IO21
- J5 pad 4: +3.3V -> /IO45
- J5 pad 5: /IO19 -> /MISO
- J5 pad 6: +BATT -> /IO41
- J5 pad 7: /IO20 -> /SCK
- J5 pad 8: GND -> /IO42
- J5 pad 9: /IO21 -> /MOSI
Routing:
- net GND: track 260.2 -> 469.6 mm, vias 7 -> 4
- net /DC: track 5.41 -> 142.8 mm, vias 1 -> 3
- net /DAT1: track 167.5 -> 44.6 mm, vias 7 -> 2
- net VBUS: track 91.6 -> 205.9 mm, vias 2 -> 4
- net /SDA: track 9.39 -> 118.9 mm, vias 0 -> 2
- net /SCK: track 152.1 -> 44.2 mm, vias 3 -> 1
- net /CS: track 6.34 -> 105.9 mm, vias 1 -> 3
- net /SCL: track 10.2 -> 108.3 mm, vias 0 -> 2
- net /EN: track 86.0 -> 179.7 mm
- net +3.3V: track 332.3 -> 257.8 mm, vias 10 -> 7
- net /IO17: track 4.94 -> 71.9 mm
- net /IO42: track 14.6 -> 79.5 mm
- net /IO18: track 8.56 -> 68.7 mm
- net Net-(U1-UD-): track 3.78 -> 63.6 mm, vias 0 -> 2
- net /IO20: track 7.34 -> 60.3 mm
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
Commit message: finish mosokik route
Parts:
- moved C17 0.48 mm to (156.6, 116.6)
- moved C16 0.28 mm to (156.6, 118.6)
Routing:
- net +3.3V: track 257.8 -> 429.3 mm, vias 7 -> 8
- net /RESET: track 22.5 -> 118.3 mm, vias 0 -> 3
- net /MOSI: track 43.0 -> 87.1 mm, vias 1 -> 3
- net /EN: track 179.7 -> 220.4 mm
- net /SCK: track 44.2 -> 80.6 mm, vias 1 -> 3
- net /IO0: track 58.7 -> 89.2 mm, vias 3 -> 2
- net /SCL: track 108.3 -> 101.0 mm
- net Net-(U1-UD-): track 63.6 -> 70.7 mm
- net Net-(U1-UD+): track 62.7 -> 68.7 mm
- net /IO42: track 79.5 -> 73.6 mm
- net /IO20: track 60.3 -> 55.3 mm
- net /DAT1: track 44.6 -> 49.2 mm
- net /~{ALRT}: track 57.6 -> 53.2 mm
- net /CS: track 105.9 -> 102.1 mm
- net /IO19: track 63.6 -> 60.0 mm
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
Commit message: generate gerbers
Routing:
- net /DAT0: track 37.3 -> 40.6 mm
- net /IO48: track 54.0 -> 51.0 mm
- net /SCL: track 101.0 -> 103.5 mm
- net /IO47: track 47.6 -> 45.2 mm
- net /EN: track 220.4 -> 218.5 mm
- net /SDA: track 115.7 -> 117.6 mm
- net /RESET: track 118.3 -> 120.1 mm
- net /CS: track 102.1 -> 103.5 mm
- net /IO45: track 60.5 -> 59.4 mm
- net /DAT1: track 49.2 -> 48.2 mm
- net +BATT: track 75.5 -> 76.4 mm
- net /IO21: track 45.2 -> 44.3 mm
- net (no net): vias 0 -> 4
Other:
- board size 60 x 60 mm -> 145.7 x 128.7 mm
